Commit message: added functionality for FR3

File: src/fairino3_v6_moveit2_config/config/fairino3_v6_robot.urdf.xacro (robot description, xacro)
@@ -7,44 +7,3 @@
     <xacro:include filename="fairino3_v6_robot.ros2_control.xacro" />
     <xacro:fairino3_v6_robot_ros2_control name="FakeSystem" initial_positions_file="$(arg initial_positions_file)"/>
-    <!-- Custom args -->
-    <!-- <xacro:arg name="gripper" default="None"/>
-    <xacro:arg name="mount" default='None'/> -->
-<!--     <xacro:if value="${$(arg gripper) == 'pgc140'}">
-        <link name="world_link">
-            <parent link="world"/>
-            <child
-        </link>
-    </xacro:if> -->
-    <!-- <xacro:if value="${$(arg mount) == 'box'}">
-        <link name="mount_link">
-            <joint name="fixed" type="fixed">
-                <parent link="mount_link"/>
-                <child link="world"/>
-            </joint>
-            <visual>
-                <geometry>
-                    <box size="1 1 1"/>
-                </geometry>
-                <material name="red">
-                    <color rgba="1 0 0 1"/>
-                </material>
-            </visual>
-            <collision>
-                <geometry>
-                    <box size="1 1 1"/>
-                </geometry>
-            </collision>
-            <inertial>
-                <mass value="1.0"/>
-                <inertia ixx="0.01" ixy="0.0" ixz="0.0" iyy="0.01" iyz="0.0" izz="0.01"/>
-            </inertial>
-        </link>
-    </xacro:if> -->
-    <!-- <xacro:if value="${$(arg mount) == 'None'}">
-        <link name="world"/>
-            <joint name="fixed" type="fixed">
-                <parent link="world"/>
-                <child link="base_link"/>
-            </joint>
-    </xacro:if> -->
 </robot>
