Commit message: first commit for SyncDemo

File: src/fairino3_v6_moveit2_config/config/fairino3_v6_robot.ros2_control.xacro (robot description, xacro)
@@ -17,12 +17,4 @@
               </xacro:if>
           </hardware>
-          <xacro:if value="${ros2_control_header != 'world'}">
-              <joint name="${ros2_control_header}_joint">
-                  <command_interface name="position"/>
-                  <state_interface name="position">
-                    <param name="initial_value">0.0</param>
-                  </state_interface>
-              </joint>
-          </xacro:if>
           <joint name="j1">
               <command_interface name="position"/>
@@ -61,4 +53,12 @@
               </state_interface>
           </joint>
+          <xacro:if value="${ros2_control_header != 'world'}">
+              <joint name="mill_to_door_joint">
+                  <command_interface name="position"/>
+                  <state_interface name="position">
+                    <param name="initial_value">0.0</param>
+                  </state_interface>
+              </joint>
+          </xacro:if>
         </ros2_control>
         <xacro:if value="${control_system == 'gazebo'}">

File: src/fairino3_v6_moveit2_config/config/fairino3_v6_robot.srdf.xacro (robot description, xacro)
@@ -13,6 +13,8 @@
     <group name="fairino3_v6_group">
         <xacro:if value="${'$(arg mount)' != 'world'}">
-            <joint name="$(arg mount)_joint" value="0.0"/>
+            <joint name="mill_to_door_joint" value="0.0"/>
         </xacro:if>
+        <!-- Temp -->
+        <joint name="roland_mill_door_joint"/>
         <joint name="j1"/>
         <joint name="j2"/>
@@ -25,5 +27,5 @@
     <!--GROUP STATES: Purpose: Define a named state for a particular group, in terms of joint values. This is useful to define states like 'folded arms'-->
     <group_state name="pos1" group="fairino3_v6_group">
-        <xacro:if value="${'$(arg mount)' != 'world'}">
+        <xacro:if value="${'rail' in '$(arg mount)'}">
             <joint name="$(arg mount)_joint" value="0.0"/>
         </xacro:if>
@@ -36,5 +38,5 @@
     </group_state>
     <group_state name="pos2" group="fairino3_v6_group">
-        <xacro:if value="${'$(arg mount)' != 'world'}">
+        <xacro:if value="${'rail' in '$(arg mount)'}">
             <joint name="$(arg mount)_joint" value="0.0"/>
         </xacro:if>

File: src/fairino5_v6_moveit2_config/config/fairino5_v6_robot.srdf.xacro (robot description, xacro)
@@ -12,5 +12,5 @@
     <xacro:arg name="mount" default="world"/>
     <group name="fairino5_v6_group">
-        <xacro:if value="${'$(arg mount)' != 'world'}">
+        <xacro:if value="${'rail' in '$(arg mount)'}">
             <joint name="$(arg mount)_joint"/>
         </xacro:if>

File: src/rail_description/config/modular_table.urdf.xacro (robot description, xacro)
@@ -27,4 +27,12 @@
       </inertial>
     </link>
+    <link name="mill_door_link">
+      <visual>
+        <geometry>
+          <box size="0.3 0.3 0.05"/>
+        </geometry>
+        <material name="blue"><color rgba="0.0 0.0 0.8 1.0"/></material>
+      </visual>
+    </link>
     <link name="modular_table_carriage"/>
     <joint name="modular_table_joint" type="fixed">

File: src/rail_description/config/sync_table2.ros2_control.xacro (robot description, xacro)
@@ -1,9 +1,9 @@
 <?xml version="1.0"?>
 <robot xmlns:xacro="http://www.ros.org/wiki/xacro">
-  <ros2_control name="RailControl" type="system">
-    <joint name="test_rail_joint">
+  <ros2_control name="MillDoorControl" type="system">
+    <joint name="mill_to_door_joint">
       <command_interface name="position">
-        <param name="min">-0.9</param>
-        <param name="max">0.9</param>
+        <param name="min">-0</param>
+        <param name="max">0.5</param>
       </command_interface>
       <state_interface name="position"/>

Commit message: Modularized sync table

File: src/fairino3_v6_moveit2_config/config/fairino3_v6_robot.ros2_control.xacro (robot description, xacro)
@@ -54,5 +54,5 @@
           </joint>
           <xacro:if value="${ros2_control_header != 'world'}">
-              <joint name="mill_to_door_joint">
+              <joint name="${ros2_control_header}_joint">
                   <command_interface name="position"/>
                   <state_interface name="position">

File: src/fairino3_v6_moveit2_config/config/fairino3_v6_robot.srdf.xacro (robot description, xacro)
@@ -13,8 +13,6 @@
     <group name="fairino3_v6_group">
         <xacro:if value="${'$(arg mount)' != 'world'}">
-            <joint name="mill_to_door_joint" value="0.0"/>
+            <joint name="$(arg mount)_joint" value="0.0"/>
         </xacro:if>
-        <!-- Temp -->
-        <joint name="roland_mill_door_joint"/>
         <joint name="j1"/>
         <joint name="j2"/>
@@ -27,5 +25,5 @@
     <!--GROUP STATES: Purpose: Define a named state for a particular group, in terms of joint values. This is useful to define states like 'folded arms'-->
     <group_state name="pos1" group="fairino3_v6_group">
-        <xacro:if value="${'rail' in '$(arg mount)'}">
+        <xacro:if value="${'$(arg mount)' != 'world'}">
             <joint name="$(arg mount)_joint" value="0.0"/>
         </xacro:if>
@@ -38,5 +36,5 @@
     </group_state>
     <group_state name="pos2" group="fairino3_v6_group">
-        <xacro:if value="${'rail' in '$(arg mount)'}">
+        <xacro:if value="${'$(arg mount)' != 'world'}">
             <joint name="$(arg mount)_joint" value="0.0"/>
         </xacro:if>

File: src/rail_description/config/sync_table2.urdf.xacro (robot description, xacro)
@@ -54,5 +54,5 @@
     </link>
     <!-- MILL TO MILL DOOR -->
-    <joint name="mill_to_door_joint" type="prismatic">
+    <joint name="sync_table2_joint" type="prismatic">
       <parent link="roland_mill_base"/>
       <child link="roland_mill_door"/>
@@ -67,5 +67,5 @@
           <mesh filename="package://rail_description/config/sync_table/RolandMillDoor.stl" scale="0.00115 0.001 0.0009"/>
         </geometry>
-        <material name="transp_grey"><color rgba="0.8 0.8 0.8 0.5"/></material>
+        <material name="transp_grey"><color rgba="0.7 0.7 0.7 0.7"/></material>
       </visual>
       <collision>
@@ -83,5 +83,5 @@
     </link>
     <link name="sync_table2_carriage"/>
-    <joint name="sync_table2_joint" type="fixed">
+    <joint name="sync_table2_mount_joint" type="fixed">
       <parent link="sync_table2_base"/>
       <child link="sync_table2_carriage"/>
