Commit message: No rail usagegit add --all

File: src/rail_description/config/test_rail.ros2_control.xacro (robot description, xacro)
@@ -8,11 +8,11 @@
                   <plugin>gz_ros2_control/GazeboSimSystem</plugin>
               </xacro:if>
-          </hardware>
-          <joint name="rail_joint">
-              <command_interface name="position"/>
-              <state_interface name="position">
-                <param name="initial_value">0.0</param>
-              </state_interface>
-          </joint>
+            </hardware>
+            <joint name="rail_joint">
+                <command_interface name="position"/>
+                <state_interface name="position">
+                    <param name="initial_value">0.0</param>
+                </state_interface>
+            </joint>
         </ros2_control>
         <xacro:if value="${'$(arg control_system)' == 'gazebo'}">
