Commit message: Added new set up

File: src/rail_description/config/sync_table2.urdf.xacro (robot description, xacro)
@@ -31,5 +31,5 @@
       <parent link="sync_table2_base"/>
       <child link="roland_mill_base"/>
-      <origin xyz="1 -0.125 0.71" rpy="0 0 -1.5707"/>
+      <origin xyz="1 0.075 0.705" rpy="0 0 -1.5707"/>
     </joint>
     <link name="roland_mill_base">
@@ -82,9 +82,9 @@
       </inertial>
     </link>
-    <!-- MILL TO SLIDER -->
+    <!-- MILL TO TRY RACK -->
     <joint name="sync_table2_slider_joint" type="fixed">
       <parent link="roland_mill_base"/>
       <child link="roland_slider"/>
-      <origin xyz="-0.05 0 0" rpy="1.57 0 4.71"/>
+      <origin xyz="0.75 0 0" rpy="1.57 0 4.71"/>
       <axis xyz="0 0 1"/>
       <limit lower="0" upper="0.5" effort="1000.0" velocity="0.5"/>
@@ -94,13 +94,55 @@
       <visual>
         <geometry>
-          <mesh filename="package://rail_description/config/sync_table/SyncSlider.stl"/>
+          <mesh filename="package://rail_description/config/sync_table/SyncTrayChassis.stl" scale="0.1 0.1 0.1"/>
         </geometry>
         <material name="grey"><color rgba="0.7 0.7 0.7 1"/></material>
       </visual>
-      <!-- <collision>
+      <inertial>
+        <mass value="0.001"/>
+        <origin xyz="0 0 0" rpy="0 0 0"/>
+        <inertia ixx="0.0001" ixy="0" ixz="0"
+                              iyy="0.0001" iyz="0"
+                                            izz="0.0001"/>
+      </inertial>
+    </link>
+    <!-- TRAY HOLDER JOINTS -->
+    <joint name="bottom_drawer_joint" type="prismatic">
+      <parent link="roland_slider"/>
+      <child link="bottom_drawer"/>
+      <origin xyz="0 0 0" rpy="0 0 0"/>
+      <axis xyz="0 1 0"/>
+      <limit lower="0" upper="0.5" effort="1000.0" velocity="0.5"/>
+      <dynamics damping="0.0" friction="0.0"/>
+    </joint>
+    <link name="bottom_drawer">
+      <visual>
         <geometry>
-          <mesh filename="package://rail_description/config/sync_table/SyncSlider.stl" scale="0.001 0.001 0.001"/>
+          <mesh filename="package://rail_description/config/sync_table/SyncBottomDrawer.stl" scale="0.1 0.1 0.1"/>
         </geometry>
-      </collision> -->
+        <material name="grey"><color rgba="0.7 0.7 0.7 1"/></material>
+      </visual>
+      <inertial>
+        <mass value="0.001"/>
+        <origin xyz="0 0 0" rpy="0 0 3.14"/>
+        <inertia ixx="0.0001" ixy="0" ixz="0"
+                              iyy="0.0001" iyz="0"
+                                            izz="0.0001"/>
+      </inertial>
+    </link>
+    <joint name="top_drawer_joint" type="prismatic">
+      <parent link="roland_slider"/>
+      <child link="top_drawer"/>
+      <origin xyz="0 0 0" rpy="0 0 0"/>
+      <axis xyz="0 1 0"/>
+      <limit lower="0" upper="0.5" effort="1000.0" velocity="0.5"/>
+      <dynamics damping="0.0" friction="0.0"/>
+    </joint>
+    <link name="top_drawer">
+      <visual>
+        <geometry>
+          <mesh filename="package://rail_description/config/sync_table/SyncTopDrawer.stl" scale="0.1 0.1 0.1"/>
+        </geometry>
+        <material name="grey"><color rgba="0.7 0.7 0.7 1"/></material>
+      </visual>
       <inertial>
         <mass value="0.001"/>
@@ -115,5 +157,5 @@
       <parent link="sync_table2_base"/>
       <child link="sync_table2_carriage"/>
-      <origin xyz="0.125 -0.3 0.7" rpy="0 0 3.14"/>
+      <origin xyz="0 -0.2 0.7" rpy="0 0 3.14"/>
     </joint>
   </xacro:macro>
