Commit message: FR5 done!

File: src/fairino5_v6_moveit2_config/config/fairino5_v6_robot.srdf.xacro (robot description, xacro)
@@ -10,6 +10,9 @@
     <!--CHAINS: When a chain is specified, all the links along the chain (including endpoints) are included in the group. Additionally, all the joints that are parents to included links are also included. This means that joints along the chain and the parent joint of the base link are included in the group-->
     <!--SUBGROUPS: Groups can also be formed by referencing to already defined group names-->
+    <xacro:arg name="mount" default="world"/>
     <group name="fairino5_v6_group">
-        <joint name="test_rail_joint"/>
+        <xacro:if value="${'$(arg mount)' != 'world'}">
+            <joint name="$(arg mount)_joint" value="0.0"/>
+        </xacro:if>
         <joint name="j1"/>
         <joint name="j2"/>
@@ -22,5 +25,7 @@
     <!--GROUP STATES: Purpose: Define a named state for a particular group, in terms of joint values. This is useful to define states like 'folded arms'-->
     <group_state name="pos1" group="fairino5_v6_group">
-        <joint name="test_rail_joint" value="0.0"/>
+        <xacro:if value="${'$(arg mount)' != 'world'}">
+            <joint name="$(arg mount)_joint" value="0.0"/>
+        </xacro:if>
         <joint name="j1" value="2.1093"/>
         <joint name="j2" value="-1.9252"/>
@@ -31,5 +36,7 @@
     </group_state>
     <group_state name="pos2" group="fairino5_v6_group">
-        <joint name="test_rail_joint" value="0.0"/>
+        <xacro:if value="${'$(arg mount)' != 'world'}">
+            <joint name="$(arg mount)_joint" value="0.0"/>
+        </xacro:if>
         <joint name="j1" value="1.0631"/>
         <joint name="j2" value="-1.6889"/>
@@ -52,6 +59,8 @@
     <disable_collisions link1="wrist2_link" link2="wrist3_link" reason="Adjacent"/>
     <!-- temp-->
-    <disable_collisions link1="base_link" link2="test_rail_base" reason="Never"/>
-    <disable_collisions link1="base_link" link2="test_rail_carriage" reason="Never"/>
-    <disable_collisions link1="test_rail_carriage" link2="test_rail_base" reason="Never"/>
+    <xacro:if value="${'$(arg mount)' != 'world'}">
+        <disable_collisions link1="base_link" link2="$(arg mount)_base" reason="Never"/>
+        <disable_collisions link1="base_link" link2="$(arg mount)_carriage" reason="Never"/>
+        <disable_collisions link1="$(arg mount)_carriage" link2="$(arg mount)_base" reason="Never"/>
+    </xacro:if>
 </robot>

File: src/fairino_description/robots/test_fairino.urdf.xacro (robot description, xacro)
@@ -12,5 +12,4 @@
     <xacro:if value="${'$(arg robot_mount)' != 'world'}">
         <xacro:include filename="$(find rail_description)/config/$(arg robot_mount).urdf.xacro"/>
-        <!-- <xacro:fairino5/> -->
         <xacro:test_rail parent="world"/>
         <joint name="robot_to_rail" type="fixed">
