Commit message: Idek anymore. Robot alone works, trying to seperate the move groups

File: src/fairino5_v6_moveit2_config/config/fairino5_v6_robot.srdf.xacro (robot description, xacro)
@@ -4,5 +4,5 @@
     A URDF file must exist for this robot as well, where the joints and the links that are referenced are defined
 -->
-<robot name="fairino5_v6_robot" xmlns:xacro="http://www.ros.org/wiki/xacro">
+<robot name="fairino_robot" xmlns:xacro="http://www.ros.org/wiki/xacro">
     <!--GROUPS: Representation of a set of joints and links. This can be useful for specifying DOF to plan for, defining arms, end effectors, etc-->
     <!--LINKS: When a link is specified, the parent joint of that link (if it exists) is automatically included-->

File: src/fairino_description/robots/test_fairino.urdf.xacro (robot description, xacro)
@@ -11,4 +11,5 @@
     <link name="world"/>
     <xacro:if value="${'$(arg robot_mount)' != 'world'}">
+        <xacro:include filename="$(find rail_description)/config/$(arg robot_mount).ros2_control.xacro"/>
         <xacro:include filename="$(find rail_description)/config/$(arg robot_mount).urdf.xacro"/>
         <xacro:call macro="$(arg robot_mount)" parent="world"/>

File: src/rail_description/config/test_rail.ros2_control.xacro (robot description, xacro)
@@ -2,4 +2,5 @@
 <robot xmlns:xacro="http://www.ros.org/wiki/xacro">
   <ros2_control name="RailControl" type="system">
+    <plugin>mock_components/GenericSystem</plugin>
     <joint name="test_rail_joint">
       <command_interface name="position">

File: src/rail_description/config/test_rail.urdf.xacro (robot description, xacro)
@@ -1,5 +1,5 @@
 <?xml version="1.0"?>
 <robot xmlns:xacro="http://www.ros.org/wiki/xacro">
-  <xacro:macro name="test_rail" params="parent length:=1.0 width:=1.0">
+  <xacro:macro name="test_rail" params="parent">
     <xacro:property name="rail_description" value="$(find fairino_gazebo_config)/config/rail_defaults.yaml"/>
     <xacro:property name="rail_rail_config" value="${xacro.load_yaml(rail_description)}"/>
