Commit message: not super sure what changed, went a bit skitz but should be stable

File: src/fairino5_v6_moveit2_config/config/fairino_v6_robot.ros2_control.xacro (robot description, xacro)
@@ -1,8 +1,8 @@
 <?xml version="1.0"?>
 <robot xmlns:xacro="http://www.ros.org/wiki/xacro">
-    <xacro:macro name="fairino20_v6_robot_ros2_control" params="name initial_positions_file ros2_control_header:=world control_system:=moveit">
+    <xacro:macro name="fairino_v6_robot_ros2_control" params="name initial_positions_file ros2_control_header:=world control_system:=moveit">
         <xacro:property name="initial_positions" value="${xacro.load_yaml(initial_positions_file)['initial_positions']}"/>
         <!-- Xacro arg for control system (Defualted to Rviz/Moveit-->
-        <xacro:property name="controllers_yaml_name" value="${'ros2_controllers.yaml' if ros2_control_header == 'world' else 'fairino20_' + ros2_control_header + '_ros2_controllers.yaml'}"/>
+        <xacro:property name="controllers_yaml_name" value="${'ros2_controllers.yaml' if 'rail' not in ros2_control_header else 'fairino_' + ros2_control_header + '_ros2_controllers.yaml'}"/>
         <ros2_control name="${name}" type="system">
             <hardware>
@@ -54,11 +54,12 @@
           </joint>
           <xacro:if value="${'rail' in ros2_control_header}">
-              <joint name="${ros2_control_header}_joint">
-                  <command_interface name="position"/>
-                  <state_interface name="position">
-                    <param name="initial_value">0.0</param>
-                  </state_interface>
-              </joint>
+            <joint name="${ros2_control_header}_joint">
+                <command_interface name="position"/>
+                <state_interface name="position">
+                  <param name="initial_value">0.0</param>
+                </state_interface>
+            </joint>
           </xacro:if>
+            <!-- If mount is not a rail (using fixed joints) then it does not need to be added to contrl xacro -->
         </ros2_control>
         <xacro:if value="${control_system == 'gazebo'}">
@@ -66,5 +67,5 @@
               <plugin filename="libign_ros2_control-system.so"
               name="gz_ros2_control::GazeboSimROS2ControlPlugin">
-                  <parameters>$(find fairino20_v6_moveit2_config)/config/ros2_controllers.yaml</parameters>
+                  <parameters>$(find fairino5_v6_moveit2_config)/config/fairino_ros2_controllers.yaml</parameters>
               </plugin>
           </gazebo>
