Commit message: HA GOT EM

File: src/fairino5_v6_moveit2_config/config/fairino_v6_robot.ros2_control.xacro (robot description, xacro)
@@ -4,5 +4,4 @@
         <xacro:property name="initial_positions" value="${xacro.load_yaml(initial_positions_file)['initial_positions']}"/>
         <!-- Xacro arg for control system (Defualted to Rviz/Moveit-->
-        <xacro:property name="controllers_yaml_name" value="${'ros2_controllers.yaml' if 'rail' not in ros2_control_header else 'fairino_' + ros2_control_header + '_ros2_controllers.yaml'}"/>
         <ros2_control name="${name}" type="system">
             <hardware>
@@ -53,12 +52,4 @@
               </state_interface>
           </joint>
-          <xacro:if value="${'rail' in ros2_control_header}">
-            <joint name="${ros2_control_header}_joint">
-                <command_interface name="position"/>
-                <state_interface name="position">
-                  <param name="initial_value">0.0</param>
-                </state_interface>
-            </joint>
-          </xacro:if>
             <!-- If mount is not a rail (using fixed joints) then it does not need to be added to contrl xacro -->
         </ros2_control>

File: src/fairino_description/robots/fairino_robot.srdf.xacro (robot description, xacro)
@@ -4,5 +4,5 @@
     <xacro:arg name="mount" default="world"/>
     <xacro:arg name="gripper" default="none"/>
-    <xacro:arg name="axes_count" default="1"/>
+    <xacro:arg name="axes_count" default="0"/>
     <xacro:property name="prefix_arg"  value="$(arg prefix)"/>
     <xacro:property name="mount_arg"  value="$(arg mount)"/>
@@ -17,6 +17,12 @@
         </xacro:if>
     </xacro:macro>
+    <xacro:macro name="build_joints_with_poses" params="count">
+        <xacro:if value="${count}">
+            <xacro:build_joints count="${count - 1}"/>
+            <joint name="${mount_arg}_joint_${count}" value="0.0"/>
+        </xacro:if>
+    </xacro:macro>
     <group name="${prefix_arg}fairino_v6_group">
-        <xacro:if value="${mount_arg != 'world'}">
+        <xacro:if value="${mount_arg != 'world' and int(num_axes) > 0}">
             <xacro:build_joints count="${num_axes}"/>
             <xacro:property name="chain_base"  value="${mount_arg}_base"/>
@@ -36,4 +42,7 @@
     <!--GROUP STATES: Purpose: Define a named state for a particular group, in terms of joint values. This is useful to define states like 'folded arms'-->
     <group_state name="pos1" group="${prefix_arg}fairino_v6_group">
+        <xacro:if value="${mount_arg != 'world' and int(num_axes) > 0}">
+            <xacro:build_joints_with_poses count="${num_axes}"/>
+        </xacro:if>
         <joint name="j1" value="2.1093"/>
         <joint name="j2" value="-1.9252"/>
@@ -47,4 +56,7 @@
     </group_state>
     <group_state name="pos2" group="${prefix_arg}fairino_v6_group">
+        <xacro:if value="${mount_arg != 'world' and int(num_axes) > 0}">
+            <xacro:build_joints_with_poses count="${num_axes}"/>
+        </xacro:if>
         <joint name="j1" value="1.0631"/>
         <joint name="j2" value="-1.6889"/>

File: src/fairino_description/robots/test_fairino.urdf.xacro (robot description, xacro)
@@ -4,5 +4,5 @@
     <xacro:arg name="robot_mount" default="world" />
     <xacro:arg name="control_system" default="moveit" />
-    <xacro:arg name="axes" default="z" />
+    <xacro:arg name="axes" default=""/>
     <xacro:property name="robot_model" value="$(arg robot_model)" />
     <xacro:property name="robot_mount_name" value="$(arg robot_mount)" />
@@ -15,9 +15,9 @@
         <xacro:include filename="$(find rail_description)/config/$(arg robot_mount).ros2_control.xacro"/>
         <xacro:include filename="$(find rail_description)/config/$(arg robot_mount).urdf.xacro"/>
-        <xacro:call macro="$(arg robot_mount)" parent="world" axes="${rail_axes}"/>
+        <xacro:call macro="$(arg robot_mount)" parent="world"/>
         <joint name="robot_to_rail" type="fixed">
             <parent link="$(arg robot_mount)_carriage"/>
             <child link="base_link"/>
-            <origin xyz="0 0 0" rpy="0 0 3.1415"/>
+            <origin xyz="0 0 0" rpy="0 0 0"/>
         </joint>
     </xacro:if>
@@ -28,52 +28,57 @@
         </joint>
     </xacro:if>
-    <xacro:include filename="$(find ${robot_config_package})/config/${robot_model}_v6_robot.ros2_control.xacro" />
+    <xacro:include filename="$(find fairino5_v6_moveit2_config)/config/fairino_v6_robot.ros2_control.xacro" />
     <xacro:if value="${robot_model == 'fairino3'}">
         <xacro:fairino3/>
-        <xacro:fairino3_v6_robot_ros2_control
+        <!-- <xacro:fairino3_v6_robot_ros2_control
             name="Fairino3_Controller"
             initial_positions_file="${initial_positions_file}"
             ros2_control_header="$(arg robot_mount)"
-            control_system="$(arg control_system)"/>
+            control_system="$(arg control_system)"/>     -->
     </xacro:if>
     <xacro:if value="${robot_model == 'fairino5'}">
         <xacro:fairino5/>
-        <xacro:fairino5_v6_robot_ros2_control
+        <!-- <xacro:fairino5_v6_robot_ros2_control
             name="Fairino5_Controller"
             initial_positions_file="${initial_positions_file}"
             ros2_control_header="$(arg robot_mount)"
-            control_system="$(arg control_system)"/>
+            control_system="$(arg control_system)"/>     -->
     </xacro:if>
     <xacro:if value="${robot_model == 'fairino10'}">
         <xacro:fairino10/>
-        <xacro:fairino10_v6_robot_ros2_control
+        <!-- <xacro:fairino10_v6_robot_ros2_control
             name="Fairino10_Controller"
             initial_positions_file="${initial_positions_file}"
             ros2_control_header="$(arg robot_mount)"
-            control_system="$(arg control_system)"/>
+            control_system="$(arg control_system)"/>   -->
     </xacro:if>
     <xacro:if value="${robot_model == 'fairino16'}">
         <xacro:fairino16/>
-        <xacro:fairino16_v6_robot_ros2_control
+        <!-- <xacro:fairino16_v6_robot_ros2_control
             name="Fairino16_Controller"
             initial_positions_file="${initial_positions_file}"
             ros2_control_header="$(arg robot_mount)"
-            control_system="$(arg control_system)"/>
+            control_system="$(arg control_system)"/>   -->
     </xacro:if>
     <xacro:if value="${robot_model == 'fairino20'}">
         <xacro:fairino20/>
-        <xacro:fairino20_v6_robot_ros2_control
+        <!-- <xacro:fairino20_v6_robot_ros2_control
             name="Fairino20_Controller"
             initial_positions_file="${initial_positions_file}"
             ros2_control_header="$(arg robot_mount)"
-            control_system="$(arg control_system)"/>
+            control_system="$(arg control_system)"/>   -->
     </xacro:if>
     <xacro:if value="${robot_model == 'fairino30'}">
         <xacro:fairino30/>
-        <xacro:fairino30_v6_robot_ros2_control
+        <!-- <xacro:fairino30_v6_robot_ros2_control
             name="Fairino30_Controller"
             initial_positions_file="${initial_positions_file}"
             ros2_control_header="$(arg robot_mount)"
-            control_system="$(arg control_system)"/>
+            control_system="$(arg control_system)"/>   -->
     </xacro:if>
+    <xacro:fairino_v6_robot_ros2_control
+        name="Fairino_Controller"
+        initial_positions_file="${initial_positions_file}"
+        ros2_control_header="$(arg robot_mount)"
+        control_system="$(arg control_system)"/>
 </robot>

File: src/rail_description/config/test_rail.ros2_control.xacro (robot description, xacro)
@@ -4,12 +4,12 @@
     <ros2_control name="${name}" type="system">
       <hardware>
-        <xacro:if value="${control_system == 'gazebo'}">
-          <plugin>gz_ros2_control/GazeboSimSystem</plugin>
-        </xacro:if>
         <xacro:if value="${control_system == 'moveit'}">
-          <plugin>mock_components/GenericSystem</plugin>
+            <plugin>mock_components/GenericSystem</plugin>
         </xacro:if>
         <xacro:if value="${control_system == 'hardware'}">
-          <plugin>rail_hardware_interface/RailSystem</plugin>  <!-- your real driver -->
+            <plugin>fairino_hardware/FairinoHardwareInterface</plugin>
+        </xacro:if>
+        <xacro:if value="${control_system == 'gazebo'}">
+            <plugin>gz_ros2_control/GazeboSimSystem</plugin>
         </xacro:if>
       </hardware>

File: src/rail_description/config/test_rail.urdf.xacro (robot description, xacro)
@@ -1,7 +1,9 @@
 <?xml version="1.0"?>
 <robot xmlns:xacro="http://www.ros.org/wiki/xacro">
-  <xacro:macro name="test_rail" params="parent:=world axes:=z">
+  <xacro:macro name="test_rail" params="parent:=world ">
     <xacro:property name="rail_description" value="$(find fairino_gazebo_config)/config/rail_defaults.yaml"/>
     <xacro:property name="test_rail_config" value="${xacro.load_yaml(rail_description)}"/>
+    <xacro:property name="axes" value="${test_rail_config['axes']}"/>
+    <xacro:property name="num_axes" value="${len(axes)}"/>
     <xacro:include filename="$(find rail_description)/config/test_rail.ros2_control.xacro"/>
     <xacro:macro name="build_joints" params="count">
@@ -75,5 +77,13 @@
       </inertial>
     </link>
-    <xacro:build_joints count="${len(axes)}"/>
+    <xacro:build_joints count="${num_axes}"/>
+    <xacro:test_rail_ros2_control num_axes="${num_axes}"/>
+    <xacro:if value="${num_axes == 0}">
+      <joint name="base_to_carriage" type="fixed">
+      <parent link="test_rail_base"/>
+      <child link="test_rail_carriage"/>
+      <origin xyz="0 0 0" rpy="0 0 0"/>
+    </joint>
+    </xacro:if>
     <link name="test_rail_carriage">
       <visual>
@@ -89,5 +99,4 @@
       </collision> -->
     </link>
-    <xacro:test_rail_ros2_control num_axes="${len(test_rail_config['axes'])}"/>
   </xacro:macro>
 </robot>
