Commit message: Figured out the command time for JointTraj, gazebo now works with SDK fluidly

File: src/fairino5_v6_moveit2_config/config/fairino5_v6_robot.ros2_control.xacro (robot description, xacro)
@@ -5,5 +5,5 @@
         <!-- Xacro arg for control system (Defualted to Rviz/Moveit-->
         <xacro:arg name="control_system" default="moveit"/>
-        <xacro:if value="${'$(arg control_system)' != 'gazebo'}">
+        <xacro:if value="${'$(arg control_system)' == 'moveit'}">
             <ros2_control name="${name}" type="system">
                 <hardware>
@@ -51,5 +51,5 @@
         </xacro:if>
         <!-- Gazebo Control system-->
-        <xacro:if value="${'$(arg control_system)' == 'gazebo'}">
+        <xacro:if value="${'$(arg control_system)' == 'gazebo' or '$(arg control_system)' != 'moveit'}">
             <ros2_control name="GazeboSimSystem" type="system">
                 <hardware>

File: src/fairino_description/urdf/fairino5_v6.urdf (robot description, URDF)
Before this commit: robot fairino5_v6_robot, 8 links, 7 joints
Links:
- link forearm_link: mass 7.6737 -> 5
- link shoulder_link: mass 4.3771 -> 8
- link upperarm_link: mass 14.458 -> 5
- link wrist1_link: mass 1.6266 -> 1.5
- link wrist2_link: mass 1.5812 -> 1.5

Commit message: Why ground plane collide?:

File: src/fairino5_v6_moveit2_config/config/fairino5_v6_robot.ros2_control.xacro (robot description, xacro)
@@ -12,4 +12,10 @@
                     <!-- <plugin>mock_components/GenericSystem</plugin> -->
                 </hardware>
+                <joint name="linear_rail_joint">
+                    <command_interface name="position"/>
+                    <state_interface name="position">
+                      <param name="initial_value">0.0</param>
+                    </state_interface>
+                </joint>
                 <joint name="j1">
                     <command_interface name="position"/>
@@ -57,4 +63,10 @@
                     <plugin>gz_ros2_control/GazeboSimSystem</plugin>
                 </hardware>
+                <joint name="linear_rail_joint">
+                    <command_interface name="position"/>
+                    <state_interface name="position">
+                      <param name="initial_value">0.0</param>
+                    </state_interface>
+                </joint>
                 <joint name="j1">
                     <command_interface name="position"/>

File: src/fairino_description/urdf/fairino5_v6.urdf (robot description, URDF)
Before this commit: robot fairino5_v6_robot, 8 links, 7 joints
Links:
- added link rail_carriage; visual box size=0.2 0.2 0.05
Joints:
- removed joint fixed
- added joint base_to_carriage: type fixed, parent rail_carriage, child base_link
- added joint linear_rail_joint: type prismatic, parent world, child rail_carriage, origin xyz=0 0 0 rpy=0 0 0, axis 1 0 0, limit lower=0.0 upper=1.5 effort=100.0 velocity=0.5

Commit message: Cleaned ros2_control.xacro for fr5; changes need to be added to all

File: src/fairino5_v6_moveit2_config/config/fairino5_v6_robot.ros2_control.xacro (robot description, xacro)
@@ -5,99 +5,59 @@
         <!-- Xacro arg for control system (Defualted to Rviz/Moveit-->
         <xacro:arg name="control_system" default="moveit"/>
-        <xacro:if value="${'$(arg control_system)' == 'moveit'}">
-            <ros2_control name="${name}" type="system">
-                <hardware>
-                    <!-- By default, set up controllers for simulation. This won't work on real hardware -->
-                    <plugin>fairino_hardware/FairinoHardwareInterface</plugin>
-                    <!-- <plugin>mock_components/GenericSystem</plugin> -->
-                </hardware>
-                <joint name="j1">
-                    <command_interface name="position"/>
-                    <state_interface name="position">
-                      <param name="initial_value">${initial_positions['j1']}</param>
-                    </state_interface>
-                </joint>
-                <joint name="j2">
-                    <command_interface name="position"/>
-                    <state_interface name="position">
-                      <param name="initial_value">${initial_positions['j2']}</param>
-                    </state_interface>
-                </joint>
-                <joint name="j3">
-                    <command_interface name="position"/>
-                    <state_interface name="position">
-                      <param name="initial_value">${initial_positions['j3']}</param>
-                    </state_interface>
-                </joint>
-                <joint name="j4">
-                    <command_interface name="position"/>
-                    <state_interface name="position">
-                      <param name="initial_value">${initial_positions['j4']}</param>
-                    </state_interface>
-                </joint>
-                <joint name="j5">
-                    <command_interface name="position"/>
-                    <state_interface name="position">
-                      <param name="initial_value">${initial_positions['j5']}</param>
-                    </state_interface>
-                </joint>
-                <joint name="j6">
-                    <command_interface name="position"/>
-                    <state_interface name="position">
-                      <param name="initial_value">${initial_positions['j6']}</param>
-                    </state_interface>
-                </joint>
-            </ros2_control>
-        </xacro:if>
-        <!-- Gazebo Control system-->
+        <xacro:arg name="robot_mount" default="world"/>
+        <!-- <xacro:if value="${'$(arg control_system)' == 'moveit'}"> -->
+        <ros2_control name="${name}" type="system">
+            <hardware>
+              <xacro:if value="${'$(arg control_system)' == 'moveit'}">
+                  <plugin>fairino_hardware/FairinoHardwareInterface</plugin>
+              </xacro:if>
+              <xacro:if value="${'$(arg control_system)' == 'gazebo'}">
+                  <plugin>gz_ros2_control/GazeboSimSystem</plugin>
+              </xacro:if>
+          </hardware>
+          <joint name="j1">
+              <command_interface name="position"/>
+              <state_interface name="position">
+                <param name="initial_value">${initial_positions['j1']}</param>
+              </state_interface>
+          </joint>
+          <joint name="j2">
+              <command_interface name="position"/>
+              <state_interface name="position">
+                <param name="initial_value">${initial_positions['j2']}</param>
+              </state_interface>
+          </joint>
+          <joint name="j3">
+              <command_interface name="position"/>
+              <state_interface name="position">
+                <param name="initial_value">${initial_positions['j3']}</param>
+              </state_interface>
+          </joint>
+          <joint name="j4">
+              <command_interface name="position"/>
+              <state_interface name="position">
+                <param name="initial_value">${initial_positions['j4']}</param>
+              </state_interface>
+          </joint>
+          <joint name="j5">
+              <command_interface name="position"/>
+              <state_interface name="position">
+                <param name="initial_value">${initial_positions['j5']}</param>
+              </state_interface>
+          </joint>
+          <joint name="j6">
+              <command_interface name="position"/>
+              <state_interface name="position">
+                <param name="initial_value">${initial_positions['j6']}</param>
+              </state_interface>
+          </joint>
+        </ros2_control>
         <xacro:if value="${'$(arg control_system)' == 'gazebo'}">
-            <ros2_control name="GazeboSimSystem" type="system">
-                <hardware>
-                    <!-- Gazebo Simulation control -->
-                    <plugin>gz_ros2_control/GazeboSimSystem</plugin>
-                </hardware>
-                <joint name="j1">
-                    <command_interface name="position"/>
-                    <state_interface name="position">
-                      <param name="initial_value">${initial_positions['j1']}</param>
-                    </state_interface>
-                </joint>
-                <joint name="j2">
-                    <command_interface name="position"/>
-                    <state_interface name="position">
-                      <param name="initial_value">${initial_positions['j2']}</param>
-                    </state_interface>
-                </joint>
-                <joint name="j3">
-                    <command_interface name="position"/>
-                    <state_interface name="position">
-                      <param name="initial_value">${initial_positions['j3']}</param>
-                    </state_interface>
-                </joint>
-                <joint name="j4">
-                    <command_interface name="position"/>
-                    <state_interface name="position">
-                      <param name="initial_value">${initial_positions['j4']}</param>
-                    </state_interface>
-                </joint>
-                <joint name="j5">
-                    <command_interface name="position"/>
-                    <state_interface name="position">
-                      <param name="initial_value">${initial_positions['j5']}</param>
-                    </state_interface>
-                </joint>
-                <joint name="j6">
-                    <command_interface name="position"/>
-                    <state_interface name="position">
-                      <param name="initial_value">${initial_positions['j6']}</param>
-                    </state_interface>
-                </joint>
-            </ros2_control>
             <gazebo>
-                <plugin filename="libign_ros2_control-system.so"
-                name="gz_ros2_control::GazeboSimROS2ControlPlugin">
-                    <parameters>$(find fairino5_v6_moveit2_config)/config/ros2_controllers.yaml</parameters>
-                </plugin>
-            </gazebo>
+              <plugin filename="libign_ros2_control-system.so"
+              name="gz_ros2_control::GazeboSimROS2ControlPlugin">
+                  <parameters>$(find fairino5_v6_moveit2_config)/config/ros2_controllers.yaml</parameters>
+              </plugin>
+          </gazebo>
         </xacro:if>
     </xacro:macro>

Commit message: Stable; mount arg can not yet be used

File: src/fairino5_v6_moveit2_config/config/fairino5_v6_robot.ros2_control.xacro (robot description, xacro)
@@ -6,5 +6,4 @@
         <xacro:arg name="control_system" default="moveit"/>
         <xacro:arg name="robot_mount" default="world"/>
-        <!-- <xacro:if value="${'$(arg control_system)' == 'moveit'}"> -->
         <ros2_control name="${name}" type="system">
             <hardware>

File: src/fairino5_v6_moveit2_config/config/fairino5_v6_robot.urdf.xacro (robot description, xacro)
@@ -6,4 +6,21 @@
     <!-- Import control_xacro -->
     <xacro:include filename="fairino5_v6_robot.ros2_control.xacro" />
+    <xacro:arg name="robot_mount" default="world" />
+    <xacro:if value="${'$(arg robot_mount)' != 'world'}">
+        <xacro:include filename="$(find rail_description)/config/$(arg robot_mount).urdf" />
+        <joint name="robot_to_mount_joint" type="fixed">
+            <parent link="$(arg robot_mount)"/>
+            <child link="base_link"/>
+            <origin xyz="0 0 0" rpy="0 0 0"/>
+        </joint>
+    </xacro:if>
+    <xacro:if value="${'$(arg robot_mount)' == 'world'}">
+        <link name="world"/>
+        <joint name="robot_to_mount_joint" type="fixed">
+            <parent link="world"/>
+            <child link="base_link"/>
+            <origin xyz="0 0 0" rpy="0 0 0"/>
+        </joint>
+    </xacro:if>
     <xacro:fairino5_v6_robot_ros2_control name="FakeSystem" initial_positions_file="$(arg initial_positions_file)"/>
 </robot>

File: src/fairino_description/urdf/fairino5_v6.urdf (robot description, URDF)
Before this commit: robot fairino5_v6_robot, 8 links, 7 joints
Links:
- removed link world
Joints:
- removed joint fixed

Commit message: using Kinova framework

File: src/fairino5_v6_moveit2_config/config/fairino5_v6_robot.ros2_control.xacro (robot description, xacro)
@@ -1,5 +1,5 @@
 <?xml version="1.0"?>
 <robot xmlns:xacro="http://www.ros.org/wiki/xacro">
-    <xacro:macro name="fairino5_v6_robot_ros2_control" params="name initial_positions_file">
+    <xacro:macro name="fairino5_v6_robot_ros2_control" params="name initial_positions_file mount">
         <xacro:property name="initial_positions" value="${xacro.load_yaml(initial_positions_file)['initial_positions']}"/>
         <!-- Xacro arg for control system (Defualted to Rviz/Moveit-->
@@ -15,7 +15,13 @@
               </xacro:if>
           </hardware>
-          <xacro:if value="${'$(arg robot_mount)' != 'world'}">
+          <xacro:if value="${mount != 'world'}">
             <xacro:include filename="$(find rail_description)/config/$(arg robot_mount).urdf" />
-            <xacro:include filename="$(find rail_description)/config/$(arg robot_mount).ros2_control.xacro" />
+            <!-- <xacro:include filename="$(find rail_description)/config/$(arg robot_mount).ros2_control.xacro" /> -->
+            <joint name="$(arg robot_mount)_joint">
+              <command_interface name="position"/>
+              <state_interface name="position">
+                <param name="initial_value">0.0</param>
+              </state_interface>
+            </joint>
           </xacro:if>
           <joint name="j1">

File: src/fairino5_v6_moveit2_config/config/fairino5_v6_robot.srdf.xacro (robot description, xacro)
@@ -4,5 +4,5 @@
     A URDF file must exist for this robot as well, where the joints and the links that are referenced are defined
 -->
-<robot name="fairino5_v6_robot">
+<robot name="fairino5_v6_robot" xmlns:xacro="http://www.ros.org/wiki/xacro">
     <!--GROUPS: Representation of a set of joints and links. This can be useful for specifying DOF to plan for, defining arms, end effectors, etc-->
     <!--LINKS: When a link is specified, the parent joint of that link (if it exists) is automatically included-->

File: src/fairino5_v6_moveit2_config/config/fairino5_v6_robot.urdf.xacro (robot description, xacro)
@@ -7,15 +7,18 @@
     <xacro:include filename="fairino5_v6_robot.ros2_control.xacro" />
     <xacro:arg name="robot_mount" default="world" />
+    <link name="world"/>
     <xacro:if value="${'$(arg robot_mount)' != 'world'}">
-        <xacro:include filename="$(find rail_description)/config/$(arg robot_mount).urdf" />
-        <xacro:include filename="$(find rail_description)/config/$(arg robot_mount).ros2_control.xacro" />
+        <xacro:include filename="$(find rail_description)/config/$(arg robot_mount).urdf"/>
+        <!-- <xacro:include filename="$(find rail_description)/config/$(arg robot_mount).ros2_control.xacro" /> -->
+        <joint name="mount_to_world" type="fixed">
+            <parent link="world"/>
+            <child link="$(arg robot_mount)_base"/>
+        </joint>
         <joint name="robot_to_mount_joint" type="fixed">
             <parent link="$(arg robot_mount)"/>
             <child link="base_link"/>
-            <origin xyz="0 0 0" rpy="0 0 0"/>
         </joint>
     </xacro:if>
     <xacro:if value="${'$(arg robot_mount)' == 'world'}">
-        <link name="world"/>
         <joint name="robot_to_mount_joint" type="fixed">
             <parent link="world"/>
@@ -24,4 +27,4 @@
         </joint>
     </xacro:if>
-    <xacro:fairino5_v6_robot_ros2_control name="FakeSystem" initial_positions_file="$(arg initial_positions_file)"/>
+    <xacro:fairino5_v6_robot_ros2_control name="FakeSystem" initial_positions_file="$(arg initial_positions_file)" mount="$(arg robot_mount)"/>
 </robot>

File: src/rail_description/config/test_rail.urdf (robot description, URDF)
Before this commit: robot test_rail, 2 links, 1 joints
Links:
- removed link world
- added link test_rail_base
Joints:
- removed joint rail_joint
- added joint test_rail_joint: type prismatic, parent test_rail_base, child test_rail, axis 1 0 0, limit lower=0.0 upper=1.5 effort=100.0 velocity=0.5
