Commit message: It's gross, but it works!

File: src/fairino5_v6_moveit2_config/config/fairino5_v6_robot.ros2_control.xacro (robot description, xacro)
@@ -1,27 +1,28 @@
 <?xml version="1.0"?>
 <robot xmlns:xacro="http://www.ros.org/wiki/xacro">
-    <xacro:macro name="fairino5_v6_robot_ros2_control" params="name initial_positions_file mount">
+    <xacro:macro name="fairino5_v6_robot_ros2_control" params="name initial_positions_file ros2_control_header">
         <xacro:property name="initial_positions" value="${xacro.load_yaml(initial_positions_file)['initial_positions']}"/>
         <!-- Xacro arg for control system (Defualted to Rviz/Moveit-->
         <xacro:arg name="control_system" default="moveit"/>
-        <xacro:arg name="robot_mount" default="world"/>
+        <xacro:property name="controllers_yaml_name" value="${'ros2_controllers.yaml' if ros2_control_header == 'world' else 'fairino5_' + ros2_control_header + '_ros2_controllers.yaml'}"/>
         <ros2_control name="${name}" type="system">
             <hardware>
               <xacro:if value="${'$(arg control_system)' == 'moveit'}">
-                  <plugin>fairino_hardware/FairinoHardwareInterface</plugin>
+                  <!-- <plugin>fairino_hardware/FairinoHardwareInterface</plugin> -->
+                  <plugin>mock_components/GenericSystem</plugin>
               </xacro:if>
               <xacro:if value="${'$(arg control_system)' == 'gazebo'}">
                   <plugin>gz_ros2_control/GazeboSimSystem</plugin>
+                  <!-- <plugin>mock_components/GenericSystem</plugin> -->
               </xacro:if>
           </hardware>
-          <xacro:if value="${mount != 'world'}">
-            <xacro:include filename="$(find rail_description)/config/$(arg robot_mount).urdf" />
-            <!-- <xacro:include filename="$(find rail_description)/config/$(arg robot_mount).ros2_control.xacro" /> -->
-            <joint name="$(arg robot_mount)_joint">
-              <command_interface name="position"/>
-              <state_interface name="position">
-                <param name="initial_value">0.0</param>
-              </state_interface>
-            </joint>
+          <xacro:if value="${ros2_control_header != 'world'}">
+              <!-- <xacro:include filename="$(find rail_description)/config/test_rail_controller.ros2_control.xacro"/> -->
+              <joint name="${ros2_control_header}_joint">
+                  <command_interface name="position"/>
+                  <state_interface name="position">
+                    <param name="initial_value">0.0</param>
+                  </state_interface>
+              </joint>
           </xacro:if>
           <joint name="j1">
@@ -66,5 +67,5 @@
               <plugin filename="libign_ros2_control-system.so"
               name="gz_ros2_control::GazeboSimROS2ControlPlugin">
-                  <parameters>$(find fairino5_v6_moveit2_config)/config/ros2_controllers.yaml</parameters>
+                  <parameters>$(find fairino5_v6_moveit2_config)/config/${controllers_yaml_name}</parameters>
               </plugin>
           </gazebo>

File: src/fairino5_v6_moveit2_config/config/fairino5_v6_robot.srdf.xacro (robot description, xacro)
@@ -11,4 +11,5 @@
     <!--SUBGROUPS: Groups can also be formed by referencing to already defined group names-->
     <group name="fairino5_v6_group">
+        <joint name="test_rail_joint"/>
         <joint name="j1"/>
         <joint name="j2"/>
@@ -21,4 +22,5 @@
     <!--GROUP STATES: Purpose: Define a named state for a particular group, in terms of joint values. This is useful to define states like 'folded arms'-->
     <group_state name="pos1" group="fairino5_v6_group">
+        <joint name="test_rail_joint" value="0.0"/>
         <joint name="j1" value="2.1093"/>
         <joint name="j2" value="-1.9252"/>
@@ -29,4 +31,5 @@
     </group_state>
     <group_state name="pos2" group="fairino5_v6_group">
+        <joint name="test_rail_joint" value="0.0"/>
         <joint name="j1" value="1.0631"/>
         <joint name="j2" value="-1.6889"/>
@@ -48,3 +51,7 @@
     <disable_collisions link1="wrist1_link" link2="wrist3_link" reason="Never"/>
     <disable_collisions link1="wrist2_link" link2="wrist3_link" reason="Adjacent"/>
+    <!-- temp-->
+    <disable_collisions link1="base_link" link2="test_rail_base" reason="Never"/>
+    <disable_collisions link1="base_link" link2="test_rail_carriage" reason="Never"/>
+    <disable_collisions link1="test_rail_carriage" link2="test_rail_base" reason="Never"/>
 </robot>

File: src/fairino5_v6_moveit2_config/config/fairino5_v6_robot.urdf.xacro (robot description, xacro)
@@ -9,17 +9,19 @@
     <link name="world"/>
     <xacro:if value="${'$(arg robot_mount)' != 'world'}">
-        <xacro:include filename="$(find rail_description)/config/$(arg robot_mount).urdf"/>
-        <!-- <xacro:include filename="$(find rail_description)/config/$(arg robot_mount).ros2_control.xacro" /> -->
-        <joint name="mount_to_world" type="fixed">
+        <xacro:include filename="$(find rail_description)/config/$(arg robot_mount).urdf.xacro"/>
+        <xacro:include filename="$(find rail_description)/config/$(arg robot_mount).ros2_control.xacro"/>
+        <xacro:test_rail parent="world" />
+        <joint name="world_to_rail" type="fixed">
             <parent link="world"/>
             <child link="$(arg robot_mount)_base"/>
         </joint>
-        <joint name="robot_to_mount_joint" type="fixed">
-            <parent link="$(arg robot_mount)"/>
+        <joint name="robot_to_rail" type="fixed">
+            <parent link="$(arg robot_mount)_carriage"/>
             <child link="base_link"/>
+            <origin xyz="0 0 0.05" rpy="0 0 0"/>
         </joint>
     </xacro:if>
     <xacro:if value="${'$(arg robot_mount)' == 'world'}">
-        <joint name="robot_to_mount_joint" type="fixed">
+        <joint name="robot_to_world_joint" type="fixed">
             <parent link="world"/>
             <child link="base_link"/>
@@ -27,4 +29,4 @@
         </joint>
     </xacro:if>
-    <xacro:fairino5_v6_robot_ros2_control name="FakeSystem" initial_positions_file="$(arg initial_positions_file)" mount="$(arg robot_mount)"/>
+    <xacro:fairino5_v6_robot_ros2_control name="FakeSystem" initial_positions_file="$(arg initial_positions_file)"/>
 </robot>

File: src/fairino_description/robots/fairino.urdf.xacro (robot description, xacro)
@@ -1,28 +1,67 @@
 <?xml version="1.0"?>
-<robot xmlns:xacro="http://ros.org/wiki/xacro" name="$(arg name)">
+<robot xmlns:xacro="http://ros.org/wiki/xacro" name="fairino_arm">
     <!-- robot name parameter -->
-    <xacro:arg name="name" default="fairino_arm" />
+    <!-- <xacro:arg name="name" default="fairino_arm" /> -->
     <!-- Arguments -->
+    <xacro:arg name="robot_model" default="fairino5" />
     <xacro:arg name="robot_mount" default="world" />
-    <xacro:arg name="robot_model" default="fairino5" />
-    <xacro:arg name="control_system" default="moveit" />
-    <!-- import main macro -->
-    <xacro:include filename="$(find fairino_description)/robots/load_robot.xacro" />
-    <!-- initial position for simulations (Mock Hardware, Gazebo) -->
-    <xacro:arg name="initial_positions_file" default="$(find ${robot_model}_v6_moveit2_config))/config/initial_positions.yaml"/>
-    <!-- convert to property to use substitution in function -->
-    <xacro:property name="initial_positions_file" default="$(arg initial_positions_file)"/>
+    <xacro:arg name="control_system" default="gazebo" />
+    <xacro:property name="robot_model" value="$(arg robot_model)" />
+    <xacro:property name="initial_positions_file" value="$(find ${robot_config_package})/config/initial_positions.yaml"/>
+    <!-- Create package variable -->
+    <xacro:property name="robot_config_package" value="$(arg robot_model)_v6_moveit2_config" />
+    <!-- Initial positions file -->
+    <xacro:property name="initial_positions_file" value="$(find ${robot_config_package})/config/initial_positions.yaml"/>
+    <xacro:include filename="$(find ${robot_config_package})/config/$(arg robot_model)_robot.xacro"/>
+    <!-- import robot description -->
+    <link name="world"/>
+    <xacro:if value="${ robot_model == 'fairino3'}">
+        <xacro:fairino3/>
+    </xacro:if>
+    <xacro:if value="${ robot_model == 'fairino5'}">
+        <xacro:fairino5/>
+    </xacro:if>
+    <xacro:if value="${ robot_model == 'fairino10'}">
+        <xacro:fairino10 />
+    </xacro:if>
+    <xacro:if value="${ robot_model == 'fairino16'}">
+        <xacro:fairino16 />
+    </xacro:if>
+    <xacro:if value="${ robot_model == 'fairino20'}">
+        <xacro:fairino20 />
+    </xacro:if>
+    <xacro:if value="${ robot_model == 'fairino30'}">
+        <xacro:fairino30 />
+    </xacro:if>
+    <xacro:if value="${'$(arg robot_mount)' != 'world'}">
+        <xacro:include filename="$(find rail_description)/config/$(arg robot_mount).urdf.xacro"/>
+        <joint name="world_to_rail" type="fixed">
+            <parent link="world"/>
+            <child link="$(arg robot_mount)_base"/>
+        </joint>
+        <joint name="robot_to_rail" type="fixed">
+            <parent link="$(arg robot_mount)_carriage"/>
+            <child link="base_link"/>
+            <origin xyz="0 0 0.05" rpy="0 0 0"/>
+        </joint>
+    </xacro:if>
+    <xacro:if value="${'$(arg robot_mount)' == 'world'}">
+        <joint name="mount_to_world" type="fixed">
+            <parent link="world"/>
+            <child link="base_link"/>
+        </joint>
+    </xacro:if>
+    <xacro:if value="${'$(arg robot_mount)' != 'world'}">
+        <xacro:include filename="$(find rail_description)/config/$(arg robot_mount).ros2_control.xacro"/>
+        <xacro:test_rail_ros2_control name="RailHardwareInterface" />
+    </xacro:if>
     <!-- create link fixed to the "world" -->
-    <link name="world" />
-    <xacro:load_robot
-        robot_model="$(arg robot_model)"
-        robot_mount="$(arg robot_mount)"
-        control_system="$(arg control_system)">
-    </xacro:load_robot>
+    <xacro:include filename="$(find ${robot_config_package}_v6_moveit2_config)/config/${robot_model}_v6_robot.ros2_control.xacro" />
+    <xacro:fairino5_v6_robot_ros2_control name="FakeSystem" initial_positions_file="$(arg initial_positions_file)"/>
     <xacro:if value="${'$(arg control_system)' == 'gazebo'}">
         <gazebo>
             <plugin filename="libign_ros2_control-system.so"
             name="gz_ros2_control::GazeboSimROS2ControlPlugin">
-                <parameters>$(find ${robot_model}_v6_moveit2_config)/config/ros2_controllers.yaml</parameters>
+                <parameters>$(find ${robot_config_package})/config/ros2_controllers.yaml</parameters>
             </plugin>
         </gazebo>

File: src/fairino_description/robots/load_robot.xacro (robot description, xacro)
@@ -1,23 +1,23 @@
 <?xml version="1.0"?>
 <robot xmlns:xacro="http://ros.org/wiki/xacro">
-  <xacro:macro name="load_robot" params="
-    robot_model
-    robot_mount
-    control_system">
-    <xacro:include filename="$(find ${robot_model}_v6_moveit2_config)/config/${robot_model}_v6_robot.ros2_control.xacro" />
-    <xacro:include filename="$(find ${robot_model}_v6_moveit2_config)/config/${robot_model}_v6_robot.urdf.xacro" />
-    <xacro:load_robot
-        initial_positions_file="${initial_positions_file}"
-        mount="${robot_mount}"
-        control_system="${control_system}">
-    </xacro:load_robot>
-    <link name="world"/>
-    <xacro:if value="${robot_mount == 'world'}">
-        <link name="${robot_model}_base"/>
-        <joint name="mount_to_world" type="fixed">
-            <parent link="world"/>
-            <child link="base_link"/>
-        </joint>
-    </xacro:if>
-    <!-- <xacro:include filename="$(find rail_description)/config/$(arg robot_mount).ros2_control.xacro" /> -->
+    <xacro:macro name="load_robot" params="
+        robot_model
+        robot_mount
+        control_system">
+        <!-- <xacro:arg name="robot_model" default="fairino5" />
+        <xacro:arg name="robot_mount" default="world" />
+        <xacro:arg name="control_system" default="moveit" /> -->
+        <xacro:include filename="$(find ${robot_model}_v6_moveit2_config)/config/${robot_model}_v6_robot.urdf.xacro" />
+        <!-- <xacro:load_robot
+            robot_model="$(arg robot_model)"
+            robot_mount="$(arg robot_mount)"
+            control_system="$(arg control_system)">
+        </xacro:load_robot> -->
+        <xacro:if value="${robot_mount == 'world'}">
+            <joint name="mount_to_world" type="fixed">
+                <parent link="world"/>
+                <child link="base_link"/>
+            </joint>
+        </xacro:if>
     </xacro:macro>
+</robot>

File: src/rail_description/config/test_rail.ros2_control.xacro (robot description, xacro)
@@ -1,27 +1,16 @@
 <?xml version="1.0"?>
 <robot xmlns:xacro="http://www.ros.org/wiki/xacro">
-    <xacro:macro name="test_rail_ros2_control" params="name">
-        <!-- Xacro arg for control system (Defualted to Rviz/Moveit-->
-        <ros2_control name="${name}" type="system">
-            <hardware>
-              <xacro:if value="${'$(arg control_system)' == 'gazebo'}">
-                  <plugin>gz_ros2_control/GazeboSimSystem</plugin>
-              </xacro:if>
-            </hardware>
-            <joint name="rail_joint">
-                <command_interface name="position"/>
-                <state_interface name="position">
-                    <param name="initial_value">0.0</param>
-                </state_interface>
-            </joint>
-        </ros2_control>
-        <xacro:if value="${'$(arg control_system)' == 'gazebo'}">
-            <gazebo>
-              <plugin filename="libign_ros2_control-system.so"
-              name="gz_ros2_control::GazeboSimROS2ControlPlugin">
-                  <parameters>$(find rail_description)/config/test_rail_controllers.yaml</parameters>
-              </plugin>
-          </gazebo>
-        </xacro:if>
-    </xacro:macro>
+  <ros2_control name="RailControl" type="system">
+    <!-- <hardware> -->
+      <!-- <plugin>gz_ros2_control/GazeboSimSystem</plugin> -->
+      <!-- <plugin>mock_components/GenericSystem</plugin> -->
+    <!-- </hardware> -->
+    <joint name="test_rail_joint">
+      <command_interface name="position">
+        <param name="min">-0.9</param>
+        <param name="max">0.9</param>
+      </command_interface>
+      <state_interface name="position"/>
+    </joint>
+  </ros2_control>
 </robot>

Commit message: demo.launch works on HW, but test_sim does not

File: src/fairino5_v6_moveit2_config/config/fairino5_v6_robot.ros2_control.xacro (robot description, xacro)
@@ -1,5 +1,5 @@
 <?xml version="1.0"?>
 <robot xmlns:xacro="http://www.ros.org/wiki/xacro">
-    <xacro:macro name="fairino5_v6_robot_ros2_control" params="name initial_positions_file ros2_control_header">
+    <xacro:macro name="fairino5_v6_robot_ros2_control" params="name initial_positions_file ros2_control_header:=world">
         <xacro:property name="initial_positions" value="${xacro.load_yaml(initial_positions_file)['initial_positions']}"/>
         <!-- Xacro arg for control system (Defualted to Rviz/Moveit-->
@@ -9,6 +9,6 @@
             <hardware>
               <xacro:if value="${'$(arg control_system)' == 'moveit'}">
-                  <!-- <plugin>fairino_hardware/FairinoHardwareInterface</plugin> -->
-                  <plugin>mock_components/GenericSystem</plugin>
+                  <plugin>fairino_hardware/FairinoHardwareInterface</plugin>
+                  <!-- <plugin>mock_components/GenericSystem</plugin> -->
               </xacro:if>
               <xacro:if value="${'$(arg control_system)' == 'gazebo'}">

Commit message: FR5 works on hardware and Gazebo

File: src/fairino5_v6_moveit2_config/config/fairino5_v6_robot.ros2_control.xacro (robot description, xacro)
@@ -1,18 +1,15 @@
 <?xml version="1.0"?>
 <robot xmlns:xacro="http://www.ros.org/wiki/xacro">
-    <xacro:macro name="fairino5_v6_robot_ros2_control" params="name initial_positions_file ros2_control_header:=world">
+    <xacro:macro name="fairino5_v6_robot_ros2_control" params="name initial_positions_file ros2_control_header:=world control_system:=moveit">
         <xacro:property name="initial_positions" value="${xacro.load_yaml(initial_positions_file)['initial_positions']}"/>
         <!-- Xacro arg for control system (Defualted to Rviz/Moveit-->
-        <xacro:arg name="control_system" default="moveit"/>
         <xacro:property name="controllers_yaml_name" value="${'ros2_controllers.yaml' if ros2_control_header == 'world' else 'fairino5_' + ros2_control_header + '_ros2_controllers.yaml'}"/>
         <ros2_control name="${name}" type="system">
             <hardware>
-              <xacro:if value="${'$(arg control_system)' == 'moveit'}">
+              <xacro:if value="${control_system != 'gazebo'}">
                   <plugin>fairino_hardware/FairinoHardwareInterface</plugin>
-                  <!-- <plugin>mock_components/GenericSystem</plugin> -->
               </xacro:if>
-              <xacro:if value="${'$(arg control_system)' == 'gazebo'}">
+              <xacro:if value="${control_system == 'gazebo'}">
                   <plugin>gz_ros2_control/GazeboSimSystem</plugin>
-                  <!-- <plugin>mock_components/GenericSystem</plugin> -->
               </xacro:if>
           </hardware>
@@ -63,5 +60,5 @@
           </joint>
         </ros2_control>
-        <xacro:if value="${'$(arg control_system)' == 'gazebo'}">
+        <xacro:if value="${control_system == 'gazebo'}">
             <gazebo>
               <plugin filename="libign_ros2_control-system.so"
