Commit message: DEPRECIATED

File: src/fairino5_v6_moveit2_config/config/fairino5_v6_robot.ros2_control.xacro (robot description, xacro)
@@ -5,111 +5,68 @@
         <!-- Xacro arg for control system (Defualted to Rviz/Moveit-->
         <xacro:arg name="control_system" default="moveit"/>
-        <xacro:if value="${'$(arg control_system)' == 'moveit'}">
-            <ros2_control name="${name}" type="system">
-                <hardware>
-                    <!-- By default, set up controllers for simulation. This won't work on real hardware -->
-                    <plugin>fairino_hardware/FairinoHardwareInterface</plugin>
-                    <!-- <plugin>mock_components/GenericSystem</plugin> -->
-                </hardware>
-                <joint name="linear_rail_joint">
-                    <command_interface name="position"/>
-                    <state_interface name="position">
-                      <param name="initial_value">0.0</param>
-                    </state_interface>
-                </joint>
-                <joint name="j1">
-                    <command_interface name="position"/>
-                    <state_interface name="position">
-                      <param name="initial_value">${initial_positions['j1']}</param>
-                    </state_interface>
-                </joint>
-                <joint name="j2">
-                    <command_interface name="position"/>
-                    <state_interface name="position">
-                      <param name="initial_value">${initial_positions['j2']}</param>
-                    </state_interface>
-                </joint>
-                <joint name="j3">
-                    <command_interface name="position"/>
-                    <state_interface name="position">
-                      <param name="initial_value">${initial_positions['j3']}</param>
-                    </state_interface>
-                </joint>
-                <joint name="j4">
-                    <command_interface name="position"/>
-                    <state_interface name="position">
-                      <param name="initial_value">${initial_positions['j4']}</param>
-                    </state_interface>
-                </joint>
-                <joint name="j5">
-                    <command_interface name="position"/>
-                    <state_interface name="position">
-                      <param name="initial_value">${initial_positions['j5']}</param>
-                    </state_interface>
-                </joint>
-                <joint name="j6">
-                    <command_interface name="position"/>
-                    <state_interface name="position">
-                      <param name="initial_value">${initial_positions['j6']}</param>
-                    </state_interface>
-                </joint>
-            </ros2_control>
-        </xacro:if>
-        <!-- Gazebo Control system-->
+        <xacro:arg name="robot_mount" default="world"/>
+        <!-- <xacro:if value="${'$(arg control_system)' == 'moveit'}"> -->
+        <ros2_control name="${name}" type="system">
+            <hardware>
+              <xacro:if value="${'$(arg control_system)' == 'moveit'}">
+                  <plugin>fairino_hardware/FairinoHardwareInterface</plugin>
+              </xacro:if>
+              <xacro:if value="${'$(arg control_system)' == 'gazebo'}">
+                  <plugin>gz_ros2_control/GazeboSimSystem</plugin>
+              </xacro:if>
+          </hardware>
+         <!-- <xacro:if value="${'$(arg robot_mount)' != 'world'}">
+              <xacro:include filename="$(find rail_description)/config/$(arg robot_mount).urdf" />
+              <joint name="$(arg robot_mount)_joint">
+                  <command_interface name="position"/>
+                  <state_interface name="position">
+                    <param name="initial_value">0.0</param>
+                  </state_interface>
+              </joint>
+          </xacro:if> -->
+          <joint name="j1">
+              <command_interface name="position"/>
+              <state_interface name="position">
+                <param name="initial_value">${initial_positions['j1']}</param>
+              </state_interface>
+          </joint>
+          <joint name="j2">
+              <command_interface name="position"/>
+              <state_interface name="position">
+                <param name="initial_value">${initial_positions['j2']}</param>
+              </state_interface>
+          </joint>
+          <joint name="j3">
+              <command_interface name="position"/>
+              <state_interface name="position">
+                <param name="initial_value">${initial_positions['j3']}</param>
+              </state_interface>
+          </joint>
+          <joint name="j4">
+              <command_interface name="position"/>
+              <state_interface name="position">
+                <param name="initial_value">${initial_positions['j4']}</param>
+              </state_interface>
+          </joint>
+          <joint name="j5">
+              <command_interface name="position"/>
+              <state_interface name="position">
+                <param name="initial_value">${initial_positions['j5']}</param>
+              </state_interface>
+          </joint>
+          <joint name="j6">
+              <command_interface name="position"/>
+              <state_interface name="position">
+                <param name="initial_value">${initial_positions['j6']}</param>
+              </state_interface>
+          </joint>
+        </ros2_control>
         <xacro:if value="${'$(arg control_system)' == 'gazebo'}">
-            <ros2_control name="GazeboSimSystem" type="system">
-                <hardware>
-                    <!-- Gazebo Simulation control -->
-                    <plugin>gz_ros2_control/GazeboSimSystem</plugin>
-                </hardware>
-                <joint name="linear_rail_joint">
-                    <command_interface name="position"/>
-                    <state_interface name="position">
-                      <param name="initial_value">0.0</param>
-                    </state_interface>
-                </joint>
-                <joint name="j1">
-                    <command_interface name="position"/>
-                    <state_interface name="position">
-                      <param name="initial_value">${initial_positions['j1']}</param>
-                    </state_interface>
-                </joint>
-                <joint name="j2">
-                    <command_interface name="position"/>
-                    <state_interface name="position">
-                      <param name="initial_value">${initial_positions['j2']}</param>
-                    </state_interface>
-                </joint>
-                <joint name="j3">
-                    <command_interface name="position"/>
-                    <state_interface name="position">
-                      <param name="initial_value">${initial_positions['j3']}</param>
-                    </state_interface>
-                </joint>
-                <joint name="j4">
-                    <command_interface name="position"/>
-                    <state_interface name="position">
-                      <param name="initial_value">${initial_positions['j4']}</param>
-                    </state_interface>
-                </joint>
-                <joint name="j5">
-                    <command_interface name="position"/>
-                    <state_interface name="position">
-                      <param name="initial_value">${initial_positions['j5']}</param>
-                    </state_interface>
-                </joint>
-                <joint name="j6">
-                    <command_interface name="position"/>
-                    <state_interface name="position">
-                      <param name="initial_value">${initial_positions['j6']}</param>
-                    </state_interface>
-                </joint>
-            </ros2_control>
             <gazebo>
-                <plugin filename="libign_ros2_control-system.so"
-                name="gz_ros2_control::GazeboSimROS2ControlPlugin">
-                    <parameters>$(find fairino5_v6_moveit2_config)/config/ros2_controllers.yaml</parameters>
-                </plugin>
-            </gazebo>
+              <plugin filename="libign_ros2_control-system.so"
+              name="gz_ros2_control::GazeboSimROS2ControlPlugin">
+                  <parameters>$(find fairino5_v6_moveit2_config)/config/ros2_controllers.yaml</parameters>
+              </plugin>
+          </gazebo>
         </xacro:if>
     </xacro:macro>

File: src/fairino5_v6_moveit2_config/config/fairino5_v6_robot.urdf.xacro (robot description, xacro)
@@ -6,4 +6,23 @@
     <!-- Import control_xacro -->
     <xacro:include filename="fairino5_v6_robot.ros2_control.xacro" />
+    <xacro:arg name="robot_mount" default="world" />
+    <link name="world"/>
+    <xacro:if value="${'$(arg robot_mount)' != 'world'}">
+        <xacro:include filename="$(find rail_description)/config/$(arg robot_mount).urdf" />
+        <joint name="mount_to_world" type="fixed">
+            <parent link="world"/>
+            <child link="$(arg robot_mount)_base"/>
+        </joint>
+        <joint name="robot_to_mount_joint" type="fixed">
+            <parent link="$(arg robot_mount)"/>
+            <child link="base_link"/>
+        </joint>
+    </xacro:if>
+    <xacro:if value="${'$(arg robot_mount)' == 'world'}">
+        <joint name="robot_to_mount_joint" type="fixed">
+            <parent link="world"/>
+            <child link="base_link"/>
+        </joint>
+    </xacro:if>
     <xacro:fairino5_v6_robot_ros2_control name="FakeSystem" initial_positions_file="$(arg initial_positions_file)"/>
 </robot>

File: src/fairino_description/urdf/fairino5_v6.urdf (robot description, URDF)
Before this commit: robot fairino5_v6_robot, 9 links, 8 joints
Links:
- removed link rail_carriage
- removed link world
Joints:
- removed joint base_to_carriage
- removed joint linear_rail_joint

Commit message: Fixed hardware and rail initial position population, still working on fixing modular table

File: src/fairino5_v6_moveit2_config/config/fairino5_v6_robot.ros2_control.xacro (robot description, xacro)
@@ -17,12 +17,4 @@
               </xacro:if>
           </hardware>
-          <xacro:if value="${ros2_control_header != 'world'}">
-              <joint name="${ros2_control_header}_joint">
-                  <command_interface name="position"/>
-                  <state_interface name="position">
-                    <param name="initial_value">0.0</param>
-                  </state_interface>
-              </joint>
-          </xacro:if>
           <joint name="j1">
               <command_interface name="position"/>
@@ -61,4 +53,12 @@
               </state_interface>
           </joint>
+          <xacro:if value="${ros2_control_header != 'world'}">
+              <joint name="${ros2_control_header}_joint">
+                  <command_interface name="position"/>
+                  <state_interface name="position">
+                    <param name="initial_value">0.0</param>
+                  </state_interface>
+              </joint>
+          </xacro:if>
         </ros2_control>
         <xacro:if value="${control_system == 'gazebo'}">

File: src/fairino5_v6_moveit2_config/config/fairino5_v6_robot.srdf.xacro (robot description, xacro)
@@ -25,5 +25,5 @@
     <!--GROUP STATES: Purpose: Define a named state for a particular group, in terms of joint values. This is useful to define states like 'folded arms'-->
     <group_state name="pos1" group="fairino5_v6_group">
-        <xacro:if value="${'$(arg mount)' != 'world'}">
+        <xacro:if value="${ 'rail' in '$(arg mount)'}">
             <joint name="$(arg mount)_joint" value="0.0"/>
         </xacro:if>
@@ -36,5 +36,5 @@
     </group_state>
     <group_state name="pos2" group="fairino5_v6_group">
-        <xacro:if value="${'$(arg mount)' != 'world'}">
+        <xacro:if value="${ 'rail' in '$(arg mount)'}">
             <joint name="$(arg mount)_joint" value="0.0"/>
         </xacro:if>

File: src/fairino_description/robots/test_fairino.urdf.xacro (robot description, xacro)
@@ -12,5 +12,5 @@
     <xacro:if value="${'$(arg robot_mount)' != 'world'}">
         <xacro:include filename="$(find rail_description)/config/$(arg robot_mount).urdf.xacro"/>
-        <xacro:test_rail parent="world"/>
+        <xacro:call macro="$(arg robot_mount)" parent="world"/>
         <joint name="robot_to_rail" type="fixed">
             <parent link="$(arg robot_mount)_carriage"/>

File: src/rail_description/config/modular_table.urdf.xacro (robot description, xacro)
@@ -1,20 +1,20 @@
 <?xml version="1.0"?>
 <robot xmlns:xacro="http://www.ros.org/wiki/xacro">
-  <xacro:macro name="test_rail" params="parent">
-    <joint name="${parent}_to_test_rail" type="fixed">
+  <xacro:macro name="modular_table" params="parent">
+    <joint name="${parent}_to_table" type="fixed">
       <parent link="${parent}"/>
-      <child link="test_rail_base"/>
+      <child link="modular_table_base"/>
       <origin xyz="0 0 0" rpy="0 0 0"/>
     </joint>
-    <link name="test_rail_base">
+    <link name="modular_table_base">
       <visual>
         <geometry>
-          <box size="2.0 0.2 0.1"/>
+          <mesh filename="package://rail_description/config/modular_table/MTDv2.STL" />
         </geometry>
         <material name="grey"><color rgba="0.5 0.5 0.5 1.0"/></material>
       </visual>
-      <!-- <collision>
+<!--       <collision>
         <geometry>
-          <box size="2.0 0.2 0.1"/>
+          <mesh filename="package://rail_description/config/modular_table/MTDv2.STL" />
         </geometry>
       </collision> -->
@@ -27,5 +27,5 @@
       </inertial>
     </link>
-    <link name="test_rail_carriage">
+    <link name="modular_table_carriage">
       <visual>
         <geometry>
@@ -34,16 +34,9 @@
         <material name="blue"><color rgba="0.0 0.0 0.8 1.0"/></material>
       </visual>
-      <!-- <collision>
-        <geometry>
-          <box size="0.3 0.3 0.05"/>
-        </geometry>
-      </collision> -->
     </link>
-    <joint name="test_rail_joint" type="prismatic">
-      <parent link="test_rail_base"/>
-      <child link="test_rail_carriage"/>
-      <axis xyz="1 0 0"/>
-      <limit lower="-0.9" upper="0.9" effort="1000.0" velocity="0.5"/>
-      <dynamics damping="10.0" friction="1.0"/>
+    <joint name="modular_table_joint" type="fixed">
+      <parent link="modular_table_base"/>
+      <child link="modular_table_carriage"/>
+      <origin xyz="0 0 0" rpy="0 0 0"/>
     </joint>
   </xacro:macro>

Commit message: Fixed table spawn

File: src/fairino5_v6_moveit2_config/config/fairino5_v6_robot.ros2_control.xacro (robot description, xacro)
@@ -4,5 +4,5 @@
         <xacro:property name="initial_positions" value="${xacro.load_yaml(initial_positions_file)['initial_positions']}"/>
         <!-- Xacro arg for control system (Defualted to Rviz/Moveit-->
-        <xacro:property name="controllers_yaml_name" value="${'ros2_controllers.yaml' if ros2_control_header == 'world' else 'fairino5_' + ros2_control_header + '_ros2_controllers.yaml'}"/>
+        <xacro:property name="controllers_yaml_name" value="${'ros2_controllers.yaml' if 'rail' not in ros2_control_header else 'fairino5_' + ros2_control_header + '_ros2_controllers.yaml'}"/>
         <ros2_control name="${name}" type="system">
             <hardware>
@@ -53,12 +53,13 @@
               </state_interface>
           </joint>
-          <xacro:if value="${ros2_control_header != 'world'}">
-              <joint name="${ros2_control_header}_joint">
-                  <command_interface name="position"/>
-                  <state_interface name="position">
-                    <param name="initial_value">0.0</param>
-                  </state_interface>
-              </joint>
+          <xacro:if value="${'rail' in ros2_control_header}">
+            <joint name="${ros2_control_header}_joint">
+                <command_interface name="position"/>
+                <state_interface name="position">
+                  <param name="initial_value">0.0</param>
+                </state_interface>
+            </joint>
           </xacro:if>
+            <!-- If mount is not a rail (using fixed joints) then it does not need to be added to contrl xacro -->
         </ros2_control>
         <xacro:if value="${control_system == 'gazebo'}">

File: src/fairino5_v6_moveit2_config/config/fairino5_v6_robot.srdf.xacro (robot description, xacro)
@@ -13,5 +13,5 @@
     <group name="fairino5_v6_group">
         <xacro:if value="${'$(arg mount)' != 'world'}">
-            <joint name="$(arg mount)_joint" value="0.0"/>
+            <joint name="$(arg mount)_joint"/>
         </xacro:if>
         <joint name="j1"/>
@@ -25,5 +25,5 @@
     <!--GROUP STATES: Purpose: Define a named state for a particular group, in terms of joint values. This is useful to define states like 'folded arms'-->
     <group_state name="pos1" group="fairino5_v6_group">
-        <xacro:if value="${ 'rail' in '$(arg mount)'}">
+        <xacro:if value="${'rail' in '$(arg mount)'}">
             <joint name="$(arg mount)_joint" value="0.0"/>
         </xacro:if>
@@ -36,5 +36,5 @@
     </group_state>
     <group_state name="pos2" group="fairino5_v6_group">
-        <xacro:if value="${ 'rail' in '$(arg mount)'}">
+        <xacro:if value="${'rail' in '$(arg mount)'}">
             <joint name="$(arg mount)_joint" value="0.0"/>
         </xacro:if>

File: src/fairino5_v6_moveit2_config/config/fairino5_v6_robot.urdf.xacro (robot description, xacro)
@@ -11,5 +11,5 @@
         <xacro:include filename="$(find rail_description)/config/$(arg robot_mount).urdf.xacro"/>
         <xacro:include filename="$(find rail_description)/config/$(arg robot_mount).ros2_control.xacro"/>
-        <xacro:test_rail parent="world" />
+        <xacro:call macro="$(arg robot_mount)" parent="world"/>
         <joint name="world_to_rail" type="fixed">
             <parent link="world"/>
@@ -19,5 +19,5 @@
             <parent link="$(arg robot_mount)_carriage"/>
             <child link="base_link"/>
-            <origin xyz="0 0 0.05" rpy="0 0 0"/>
+            <origin xyz="0 0 0.0" rpy="0 0 0"/>
         </joint>
     </xacro:if>

File: src/fairino_description/robots/test_fairino.urdf.xacro (robot description, xacro)
@@ -16,5 +16,5 @@
             <parent link="$(arg robot_mount)_carriage"/>
             <child link="base_link"/>
-            <origin xyz="0 0 0.05" rpy="0 0 0"/>
+            <origin xyz="0 0 0" rpy="0 0 3.1415"/>
         </joint>
     </xacro:if>

File: src/rail_description/config/modular_table.urdf.xacro (robot description, xacro)
@@ -5,5 +5,5 @@
       <parent link="${parent}"/>
       <child link="modular_table_base"/>
-      <origin xyz="0 0 0" rpy="0 0 0"/>
+      <origin xyz="0 0 0" rpy="0  0 0"/>
     </joint>
     <link name="modular_table_base">
@@ -14,5 +14,5 @@
         <material name="grey"><color rgba="0.5 0.5 0.5 1.0"/></material>
       </visual>
-<!--       <collision>
+      <!-- <collision>
         <geometry>
           <mesh filename="package://rail_description/config/modular_table/MTDv2.STL" />
@@ -28,15 +28,18 @@
     </link>
     <link name="modular_table_carriage">
-      <visual>
+      <!-- <visual>
         <geometry>
           <box size="0.3 0.3 0.05"/>
         </geometry>
-        <material name="blue"><color rgba="0.0 0.0 0.8 1.0"/></material>
-      </visual>
+      </visual> -->
+      <!-- <collision>
+        <geometry>
+          <box size="0.3 0.3 0.05"/>
+        </geometry>
+      </collision> -->
     </link>
     <joint name="modular_table_joint" type="fixed">
       <parent link="modular_table_base"/>
       <child link="modular_table_carriage"/>
-      <origin xyz="0 0 0" rpy="0 0 0"/>
     </joint>
   </xacro:macro>

Commit message: Fixed controller spawning

File: src/fairino5_v6_moveit2_config/config/fairino5_v6_robot.ros2_control.xacro (robot description, xacro)
@@ -4,5 +4,6 @@
         <xacro:property name="initial_positions" value="${xacro.load_yaml(initial_positions_file)['initial_positions']}"/>
         <!-- Xacro arg for control system (Defualted to Rviz/Moveit-->
-        <xacro:property name="controllers_yaml_name" value="${'ros2_controllers.yaml' if 'rail' not in ros2_control_header else 'fairino5_' + ros2_control_header + '_ros2_controllers.yaml'}"/>
+        <!-- <xacro:property name="controllers_yaml_name" value="${'ros2_controllers.yaml' if 'rail' not in ros2_control_header else 'fairino5_' + ros2_control_header + '_ros2_controllers.yaml'}"/>      -->
+        <xacro:property name="controllers_yaml_name" value="ros2_controllers.yaml"/>
         <ros2_control name="${name}" type="system">
             <hardware>

File: src/fairino_description/robots/test_fairino.urdf.xacro (robot description, xacro)
@@ -37,5 +37,5 @@
         <xacro:fairino5/>
         <xacro:fairino5_v6_robot_ros2_control
-            name="FakeSystem"
+            name="Fairino5_Controller"
             initial_positions_file="${initial_positions_file}"
             ros2_control_header="$(arg robot_mount)"
@@ -45,5 +45,5 @@
         <xacro:fairino10/>
         <xacro:fairino10_v6_robot_ros2_control
-            name="FakeSystem"
+            name="Fairino10_Controller"
             initial_positions_file="${initial_positions_file}"
             ros2_control_header="$(arg robot_mount)"
@@ -53,5 +53,5 @@
         <xacro:fairino16/>
         <xacro:fairino16_v6_robot_ros2_control
-            name="FakeSystem"
+            name="Fairino16_Controller"
             initial_positions_file="${initial_positions_file}"
             ros2_control_header="$(arg robot_mount)"
@@ -61,5 +61,5 @@
         <xacro:fairino20/>
         <xacro:fairino20_v6_robot_ros2_control
-            name="FakeSystem"
+            name="Fairino20_Controller"
             initial_positions_file="${initial_positions_file}"
             ros2_control_header="$(arg robot_mount)"
@@ -69,5 +69,5 @@
         <xacro:fairino30/>
         <xacro:fairino30_v6_robot_ros2_control
-            name="FakeSystem"
+            name="Fairino30_Controller"
             initial_positions_file="${initial_positions_file}"
             ros2_control_header="$(arg robot_mount)"
