Commit message: CHAT I DID THE THING

File: src/fairino5_v6_moveit2_config/config/fairino5_v6_robot.ros2_control.xacro (robot description, xacro)
@@ -54,5 +54,5 @@
               </state_interface>
           </joint>
-          <xacro:if value="${'rail' in ros2_control_header}">
+          <!-- <xacro:if value="${'rail' in ros2_control_header}">
             <joint name="${ros2_control_header}_joint">
                 <command_interface name="position"/>
@@ -61,5 +61,5 @@
                 </state_interface>
             </joint>
-          </xacro:if>
+          </xacro:if> -->
             <!-- If mount is not a rail (using fixed joints) then it does not need to be added to contrl xacro -->
         </ros2_control>

File: src/rail_description/config/test_rail.ros2_control.xacro (robot description, xacro)
@@ -1,13 +1,24 @@
 <?xml version="1.0"?>
 <robot xmlns:xacro="http://www.ros.org/wiki/xacro">
-  <ros2_control name="RailControl" type="system">
-    <plugin>mock_components/GenericSystem</plugin>
-    <joint name="test_rail_joint">
-      <command_interface name="position">
-        <param name="min">-0.9</param>
-        <param name="max">0.9</param>
-      </command_interface>
-      <state_interface name="position"/>
-    </joint>
-  </ros2_control>
+  <xacro:macro name="test_rail_ros2_control" params="name:=test_rail control_system:=moveit">
+    <ros2_control name="${name}" type="system">
+      <hardware>
+        <xacro:if value="${control_system == 'gazebo'}">
+          <plugin>gz_ros2_control/GazeboSimSystem</plugin>
+        </xacro:if>
+        <xacro:if value="${control_system == 'moveit'}">
+          <plugin>mock_components/GenericSystem</plugin>
+        </xacro:if>
+        <xacro:if value="${control_system == 'hardware'}">
+          <plugin>rail_hardware_interface/RailSystem</plugin>  <!-- your real driver -->
+        </xacro:if>
+      </hardware>
+      <joint name="test_rail_joint">
+        <command_interface name="position"/>
+        <state_interface name="position">
+          <param name="initial_value">0.0</param>
+        </state_interface>
+      </joint>
+    </ros2_control>
+  </xacro:macro>
 </robot>

File: src/rail_description/config/test_rail.urdf.xacro (robot description, xacro)
@@ -4,4 +4,6 @@
     <xacro:property name="rail_description" value="$(find fairino_gazebo_config)/config/rail_defaults.yaml"/>
     <xacro:property name="rail_rail_config" value="${xacro.load_yaml(rail_description)}"/>
+    <xacro:include filename="$(find rail_description)/config/test_rail.ros2_control.xacro"/>
+    <xacro:test_rail_ros2_control/>
     <joint name="${parent}_to_test_rail" type="fixed">
       <parent link="${parent}"/>
