Commit message: updated to FR5

File: src/fairino5_v6_moveit2_config/config/fairino5_robot.xacro (robot description, xacro)
@@ -456,4 +456,44 @@
             k_velocity="10" />
         </joint>
+            <link
+    name="Gripper">
+        <origin
+            xyz="0 0 0"
+            rpy="0 0 0" />
+        <mass
+            value="0.53877" />
+        <inertia
+            ixx="0.00028785"
+            ixy="-2.0584E-09"
+            ixz="-1.3892E-07"
+            iyy="0.00028896"
+            iyz="1.8115E-07"
+            izz="0.00042655" />
+        <visual>
+            <origin
+                xyz="0 0 0.102"
+                rpy="0 0 0" />
+            <geometry>
+                <mesh
+                filename="package://fairino_description/meshes/fairino3_v6/SyncGripper.STL" scale="0.1 0.1 0.1"/>
+            </geometry>
+            <material
+                name="">
+                <color
+                rgba="0.89804 0.91765 0.92941 1" />
+            </material>
+        </visual>
+    </link>
+        <joint
+            name="gripper_joint"
+            type="fixed">
+            <origin
+            xyz="0 0 0"
+            rpy="0 0 0" />
+            <parent
+            link="wrist3_link" />
+            <child
+            link="Gripper" />
+        </joint>
     </xacro:macro>
 </robot>

File: src/fairino5_v6_moveit2_config/config/fairino5_v6_robot.ros2_control.xacro (robot description, xacro)
@@ -54,11 +54,11 @@
               </state_interface>
           </joint>
-          <xacro:if value="${'rail' in ros2_control_header}">
-            <joint name="${ros2_control_header}_joint">
-                <command_interface name="position"/>
-                <state_interface name="position">
-                  <param name="initial_value">0.0</param>
-                </state_interface>
-            </joint>
+          <xacro:if value="${ros2_control_header != 'world'}">
+              <joint name="${ros2_control_header}_joint">
+                  <command_interface name="position"/>
+                  <state_interface name="position">
+                    <param name="initial_value">0.0</param>
+                  </state_interface>
+              </joint>
           </xacro:if>
             <!-- If mount is not a rail (using fixed joints) then it does not need to be added to contrl xacro -->

File: src/fairino5_v6_moveit2_config/config/fairino_v6_robot.ros2_control.xacro (robot description, xacro)
@@ -53,11 +53,11 @@
               </state_interface>
           </joint>
-          <xacro:if value="${'rail' in ros2_control_header}">
-            <joint name="${ros2_control_header}_joint">
-                <command_interface name="position"/>
-                <state_interface name="position">
-                  <param name="initial_value">0.0</param>
-                </state_interface>
-            </joint>
+          <xacro:if value="${ros2_control_header != 'world'}">
+              <joint name="${ros2_control_header}_joint">
+                  <command_interface name="position"/>
+                  <state_interface name="position">
+                    <param name="initial_value">0.0</param>
+                  </state_interface>
+              </joint>
           </xacro:if>
             <!-- If mount is not a rail (using fixed joints) then it does not need to be added to contrl xacro -->

Commit message: Fixed controlres to add tay rack

File: src/fairino5_v6_moveit2_config/config/fairino5_robot.xacro (robot description, xacro)
@@ -456,33 +456,33 @@
             k_velocity="10" />
         </joint>
-            <link
-    name="Gripper">
-        <origin
-            xyz="0 0 0"
-            rpy="0 0 0" />
-        <mass
-            value="0.53877" />
-        <inertia
-            ixx="0.00028785"
-            ixy="-2.0584E-09"
-            ixz="-1.3892E-07"
-            iyy="0.00028896"
-            iyz="1.8115E-07"
-            izz="0.00042655" />
-        <visual>
-            <origin
-                xyz="0 0 0.102"
-                rpy="0 0 0" />
-            <geometry>
-                <mesh
-                filename="package://fairino_description/meshes/fairino3_v6/SyncGripper.STL" scale="0.1 0.1 0.1"/>
-            </geometry>
-            <material
-                name="">
-                <color
-                rgba="0.89804 0.91765 0.92941 1" />
-            </material>
-        </visual>
-    </link>
+        <link
+            name="Gripper">
+            <origin
+                xyz="0 0 0"
+                rpy="0 0 0" />
+            <mass
+                value="0.53877" />
+            <inertia
+                ixx="0.00028785"
+                ixy="-2.0584E-09"
+                ixz="-1.3892E-07"
+                iyy="0.00028896"
+                iyz="1.8115E-07"
+                izz="0.00042655" />
+            <visual>
+                <origin
+                    xyz="0 0 0.102"
+                    rpy="0 0 0" />
+                <geometry>
+                    <mesh
+                    filename="package://fairino_description/meshes/fairino3_v6/SyncGripper.STL" scale="0.1 0.1 0.1"/>
+                </geometry>
+                <material
+                    name="">
+                    <color
+                    rgba="0.89804 0.91765 0.92941 1" />
+                </material>
+            </visual>
+        </link>
         <joint
             name="gripper_joint"
@@ -490,5 +490,5 @@
             <origin
             xyz="0 0 0"
-            rpy="0 0 0" />
+            rpy="0 0 1.8326" />
             <parent
             link="wrist3_link" />

File: src/fairino5_v6_moveit2_config/config/fairino5_v6_robot.ros2_control.xacro (robot description, xacro)
@@ -62,4 +62,20 @@
               </joint>
           </xacro:if>
+          <xacro:if value="${'sync' in ros2_control_header}">
+              <joint name="top_drawer_joint">
+                  <command_interface name="position"/>
+                  <state_interface name="position">
+                    <param name="initial_value">0.0</param>
+                  </state_interface>
+              </joint>
+          </xacro:if>
+          <xacro:if value="${'sync' in ros2_control_header}">
+              <joint name="bottom_drawer_joint">
+                  <command_interface name="position"/>
+                  <state_interface name="position">
+                    <param name="initial_value">0.0</param>
+                  </state_interface>
+              </joint>
+          </xacro:if>
             <!-- If mount is not a rail (using fixed joints) then it does not need to be added to contrl xacro -->
         </ros2_control>

File: src/fairino5_v6_moveit2_config/config/fairino_v6_robot.ros2_control.xacro (robot description, xacro)
@@ -61,4 +61,18 @@
               </joint>
           </xacro:if>
+          <xacro:if value="${'sync' in ros2_control_header}">
+              <joint name="top_drawer_joint">
+                  <command_interface name="position"/>
+                  <state_interface name="position">
+                    <param name="initial_value">0.0</param>
+                  </state_interface>
+              </joint>
+               <joint name="bottom_drawer_joint">
+                  <command_interface name="position"/>
+                  <state_interface name="position">
+                    <param name="initial_value">0.0</param>
+                  </state_interface>
+              </joint>
+          </xacro:if>
             <!-- If mount is not a rail (using fixed joints) then it does not need to be added to contrl xacro -->
         </ros2_control>

File: src/rail_description/config/sync_table2.urdf.xacro (robot description, xacro)
@@ -59,5 +59,5 @@
       <origin xyz="0.4175 -0.35 0.73" rpy="5.93403 0 0"/>
       <axis xyz="0 0 1"/>
-      <limit lower="0" upper="0.5" effort="1000.0" velocity="0.5"/>
+      <limit lower="0" upper="0.4" effort="100.0" velocity="0.5"/>
       <dynamics damping="0.0" friction="0.0"/>
     </joint>
@@ -111,5 +111,5 @@
       <child link="bottom_drawer"/>
       <origin xyz="0 0 0" rpy="0 0 0"/>
-      <axis xyz="0 1 0"/>
+      <axis xyz="1 0 0"/>
       <limit lower="0" upper="0.5" effort="1000.0" velocity="0.5"/>
       <dynamics damping="0.0" friction="0.0"/>
@@ -134,5 +134,5 @@
       <child link="top_drawer"/>
       <origin xyz="0 0 0" rpy="0 0 0"/>
-      <axis xyz="0 1 0"/>
+      <axis xyz="1 0 0"/>
       <limit lower="0" upper="0.5" effort="1000.0" velocity="0.5"/>
       <dynamics damping="0.0" friction="0.0"/>
@@ -157,5 +157,5 @@
       <parent link="sync_table2_base"/>
       <child link="sync_table2_carriage"/>
-      <origin xyz="0 -0.2 0.7" rpy="0 0 3.14"/>
+      <origin xyz="0 -0.2 0.7" rpy="0 0 -1.57"/>
     </joint>
   </xacro:macro>

Commit message: Small touch ups

File: src/fairino5_v6_moveit2_config/config/fairino5_robot.xacro (robot description, xacro)
@@ -490,5 +490,5 @@
             <origin
             xyz="0 0 0"
-            rpy="0 0 1.8326" />
+            rpy="0 0 -1.309" />
             <parent
             link="wrist3_link" />

File: src/rail_description/config/sync_table2.urdf.xacro (robot description, xacro)
@@ -86,5 +86,5 @@
       <parent link="roland_mill_base"/>
       <child link="roland_slider"/>
-      <origin xyz="0.75 0 0" rpy="1.57 0 4.71"/>
+      <origin xyz="0.75 -0.025 0" rpy="1.57 0 4.71"/>
       <axis xyz="0 0 1"/>
       <limit lower="0" upper="0.5" effort="1000.0" velocity="0.5"/>

Commit message: Small cahnges:

File: src/fairino5_v6_moveit2_config/config/fairino5_robot.xacro (robot description, xacro)
@@ -479,7 +479,7 @@
                 </geometry>
                 <material
-                    name="">
+                    name="grey">
                     <color
-                    rgba="0.89804 0.91765 0.92941 1" />
+                    rgba="0.7 0.7 0.7 1" />
                 </material>
             </visual>

File: src/rail_description/config/sync_table2.urdf.xacro (robot description, xacro)
@@ -96,5 +96,5 @@
           <mesh filename="package://rail_description/config/sync_table/SyncTrayChassis.stl" scale="0.1 0.1 0.1"/>
         </geometry>
-        <material name="grey"><color rgba="0.7 0.7 0.7 1"/></material>
+        <material name="dark-grey"><color rgba="0.2 0.2 0.2 1"/></material>
       </visual>
       <inertial>
@@ -112,5 +112,5 @@
       <origin xyz="0 0 0" rpy="0 0 0"/>
       <axis xyz="1 0 0"/>
-      <limit lower="0" upper="0.5" effort="1000.0" velocity="0.5"/>
+      <limit lower="0" upper="0.5" effort="100.0" velocity="0.5"/>
       <dynamics damping="0.0" friction="0.0"/>
     </joint>
@@ -135,5 +135,5 @@
       <origin xyz="0 0 0" rpy="0 0 0"/>
       <axis xyz="1 0 0"/>
-      <limit lower="0" upper="0.5" effort="1000.0" velocity="0.5"/>
+      <limit lower="0" upper="0.5" effort="100.0" velocity="0.5"/>
       <dynamics damping="0.0" friction="0.0"/>
     </joint>
