Commit message: Got env spawn to work

File: src/fairino_description/robots/fairino_robot.srdf.xacro (robot description, xacro)
@@ -1,17 +1,16 @@
 <?xml version="1.0" encoding="UTF-8"?>
-<!--This does not replace URDF, and is not an extension of URDF.
-    This is a format for representing semantic information about the robot structure.
-    A URDF file must exist for this robot as well, where the joints and the links that are referenced are defined
--->
-<robot name="fairino5_robot" xmlns:xacro="http://www.ros.org/wiki/xacro">
-    <!--GROUPS: Representation of a set of joints and links. This can be useful for specifying DOF to plan for, defining arms, end effectors, etc-->
-    <!--LINKS: When a link is specified, the parent joint of that link (if it exists) is automatically included-->
-    <!--JOINTS: When a joint is specified, the child link of that joint (which will always exist) is automatically included-->
-    <!--CHAINS: When a chain is specified, all the links along the chain (including endpoints) are included in the group. Additionally, all the joints that are parents to included links are also included. This means that joints along the chain and the parent joint of the base link are included in the group-->
-    <!--SUBGROUPS: Groups can also be formed by referencing to already defined group names-->
+<robot name="fairino_robot" xmlns:xacro="http://www.ros.org/wiki/xacro">
+    <xacro:arg name="prefix" default=""/>
     <xacro:arg name="mount" default="world"/>
-    <group name="fairino5_v6_group">
-        <xacro:if value="${'$(arg mount)' != 'world'}">
+    <xacro:arg name="gripper" default="none"/>
+    <xacro:property name="prefix_arg"  value="$(arg prefix)"/>
+    <xacro:property name="mount_arg"  value="$(arg mount)"/>
+    <xacro:property name="gripper_arg"  value="$(arg gripper)"/>
+    <xacro:property name="chain_base"  value="base_link"/>
+    <xacro:property name="chain_end"  value="wrist3_link"/>
+    <group name="${prefix_arg}fairino_v6_group">
+        <xacro:if value="${mount_arg != 'world'}">
             <joint name="$(arg mount)_joint"/>
+            <xacro:property name="chain_base"  value="$(arg mount)_base"/>
         </xacro:if>
         <joint name="j1"/>
@@ -21,9 +20,13 @@
         <joint name="j5"/>
         <joint name="j6"/>
-        <chain base_link="base_link" tip_link="wrist3_link"/>
+        <xacro:if value="${gripper_arg != 'none'}">
+            <joint name="$(arg gripper)_joint" value="0.0"/>
+            <xacro:property name="chain_end"  value="$(arg gripper)_end_link"/>
+        </xacro:if>
+        <chain base_link="${chain_base}" tip_link="${chain_end}"/>
     </group>
     <!--GROUP STATES: Purpose: Define a named state for a particular group, in terms of joint values. This is useful to define states like 'folded arms'-->
-    <group_state name="pos1" group="fairino5_v6_group">
-        <xacro:if value="${'$(arg mount)' != 'world'}">
+    <group_state name="pos1" group="${prefix_arg}fairino_v6_group">
+        <xacro:if value="${mount_arg != 'world'}">
             <joint name="$(arg mount)_joint" value="0.0"/>
         </xacro:if>
@@ -34,7 +37,10 @@
         <joint name="j5" value="-1.4343"/>
         <joint name="j6" value="0"/>
+        <xacro:if value="${gripper_arg != 'none'}">
+            <joint name="$(arg gripper)_joint" value="0.0"/>
+        </xacro:if>
     </group_state>
-    <group_state name="pos2" group="fairino5_v6_group">
-        <xacro:if value="${'$(arg mount)' != 'world'}">
+    <group_state name="pos2" group="${prefix_arg}fairino_v6_group">
+        <xacro:if value="${mount_arg != 'world'}">
             <joint name="$(arg mount)_joint" value="0.0"/>
         </xacro:if>
@@ -45,4 +51,7 @@
         <joint name="j5" value="-1.5018"/>
         <joint name="j6" value="0"/>
+        <xacro:if value="${gripper_arg != 'none'}">
+            <joint name="$(arg gripper)_joint" value="0.0"/>
+        </xacro:if>
     </group_state>
     <!--DISABLE COLLISIONS: By default it is assumed that any link of the robot could potentially come into collision with any other link in the robot. This tag disables collision checking between a specified pair of links. -->
@@ -59,5 +68,5 @@
     <disable_collisions link1="wrist2_link" link2="wrist3_link" reason="Adjacent"/>
     <!-- temp-->
-    <xacro:if value="${'$(arg mount)' != 'world'}">
+    <xacro:if value="${mount_arg != 'world'}">
         <disable_collisions link1="base_link" link2="$(arg mount)_base" reason="Never"/>
         <disable_collisions link1="base_link" link2="$(arg mount)_carriage" reason="Never"/>

Commit message: Close enough

File: src/fairino_description/robots/fairino_robot.srdf.xacro (robot description, xacro)
@@ -4,13 +4,21 @@
     <xacro:arg name="mount" default="world"/>
     <xacro:arg name="gripper" default="none"/>
+    <xacro:arg name="axes_count" default="1"/>
     <xacro:property name="prefix_arg"  value="$(arg prefix)"/>
     <xacro:property name="mount_arg"  value="$(arg mount)"/>
     <xacro:property name="gripper_arg"  value="$(arg gripper)"/>
+    <xacro:property name="num_axes"  value="$(arg axes_count)"/>
     <xacro:property name="chain_base"  value="base_link"/>
     <xacro:property name="chain_end"  value="wrist3_link"/>
+    <xacro:macro name="build_joints" params="count">
+        <xacro:if value="${count}">
+            <xacro:build_joints count="${count - 1}"/>
+            <joint name="${mount_arg}_joint_${count}"/>
+        </xacro:if>
+    </xacro:macro>
     <group name="${prefix_arg}fairino_v6_group">
         <xacro:if value="${mount_arg != 'world'}">
-            <joint name="$(arg mount)_joint"/>
-            <xacro:property name="chain_base"  value="$(arg mount)_base"/>
+            <xacro:build_joints count="${num_axes}"/>
+            <xacro:property name="chain_base"  value="${mount_arg}_base"/>
         </xacro:if>
         <joint name="j1"/>
@@ -28,7 +36,4 @@
     <!--GROUP STATES: Purpose: Define a named state for a particular group, in terms of joint values. This is useful to define states like 'folded arms'-->
     <group_state name="pos1" group="${prefix_arg}fairino_v6_group">
-        <xacro:if value="${mount_arg != 'world'}">
-            <joint name="$(arg mount)_joint" value="0.0"/>
-        </xacro:if>
         <joint name="j1" value="2.1093"/>
         <joint name="j2" value="-1.9252"/>
@@ -42,7 +47,4 @@
     </group_state>
     <group_state name="pos2" group="${prefix_arg}fairino_v6_group">
-        <xacro:if value="${mount_arg != 'world'}">
-            <joint name="$(arg mount)_joint" value="0.0"/>
-        </xacro:if>
         <joint name="j1" value="1.0631"/>
         <joint name="j2" value="-1.6889"/>

File: src/fairino_description/robots/test_fairino.urdf.xacro (robot description, xacro)
@@ -4,6 +4,8 @@
     <xacro:arg name="robot_mount" default="world" />
     <xacro:arg name="control_system" default="moveit" />
+    <xacro:arg name="axes" default="z" />
     <xacro:property name="robot_model" value="$(arg robot_model)" />
     <xacro:property name="robot_mount_name" value="$(arg robot_mount)" />
+    <xacro:property name="rail_axes" value="$(arg axes)" />
     <xacro:property name="robot_config_package" value="${robot_model}_v6_moveit2_config" />
     <xacro:property name="initial_positions_file" value="$(find ${robot_config_package})/config/initial_positions.yaml"/>
@@ -13,5 +15,5 @@
         <xacro:include filename="$(find rail_description)/config/$(arg robot_mount).ros2_control.xacro"/>
         <xacro:include filename="$(find rail_description)/config/$(arg robot_mount).urdf.xacro"/>
-        <xacro:call macro="$(arg robot_mount)" parent="world"/>
+        <xacro:call macro="$(arg robot_mount)" parent="world" axes="${rail_axes}"/>
         <joint name="robot_to_rail" type="fixed">
             <parent link="$(arg robot_mount)_carriage"/>

File: src/rail_description/config/test_rail.ros2_control.xacro (robot description, xacro)
@@ -1,5 +1,5 @@
 <?xml version="1.0"?>
 <robot xmlns:xacro="http://www.ros.org/wiki/xacro">
-  <xacro:macro name="test_rail_ros2_control" params="name:=test_rail control_system:=moveit">
+  <xacro:macro name="test_rail_ros2_control" params="name:=test_rail control_system:=moveit num_axes:=1">
     <ros2_control name="${name}" type="system">
       <hardware>
@@ -14,10 +14,17 @@
         </xacro:if>
       </hardware>
-      <joint name="test_rail_joint">
-        <command_interface name="position"/>
-        <state_interface name="position">
-          <param name="initial_value">0.0</param>
-        </state_interface>
-      </joint>
+      <xacro:macro name="build_links" params="count">
+        <xacro:if value="${count}">
+          <!-- Call macro recursively with decreased count -->
+          <xacro:build_links count="${count - 1}" />
+          <joint name="test_rail_joint_${count}">
+            <command_interface name="position"/>
+            <state_interface name="position">
+              <param name="initial_value">0.0</param>
+            </state_interface>
+          </joint>
+        </xacro:if>
+      </xacro:macro>
+      <xacro:build_links count="${num_axes}"/>
     </ros2_control>
   </xacro:macro>

File: src/rail_description/config/test_rail.urdf.xacro (robot description, xacro)
@@ -1,9 +1,53 @@
 <?xml version="1.0"?>
 <robot xmlns:xacro="http://www.ros.org/wiki/xacro">
-  <xacro:macro name="test_rail" params="parent">
+  <xacro:macro name="test_rail" params="parent:=world axes:=z">
     <xacro:property name="rail_description" value="$(find fairino_gazebo_config)/config/rail_defaults.yaml"/>
-    <xacro:property name="rail_rail_config" value="${xacro.load_yaml(rail_description)}"/>
+    <xacro:property name="test_rail_config" value="${xacro.load_yaml(rail_description)}"/>
     <xacro:include filename="$(find rail_description)/config/test_rail.ros2_control.xacro"/>
-    <xacro:test_rail_ros2_control/>
+    <xacro:macro name="build_joints" params="count">
+      <xacro:if value="${count}">
+        <!-- Call macro recursively with decreased count -->
+        <xacro:build_joints count="${count - 1}"/>
+        <!-- SET UP DEFAULTS -->
+        <xacro:property name="joint_parent" value="test_rail_link_${count}"/>
+        <xacro:property name="joint_child" value="test_rail_link_${count-1}"/>
+        <xacro:property name="axis_control" value="0 0 0"/>
+        <xacro:property name="lower_limit" value="0"/>
+        <xacro:property name="upper_limit" value="0"/>
+        <xacro:if value="${count == len(axes)}">
+          <xacro:property name="joint_parent" value="test_rail_base"/>
+        </xacro:if>
+        <xacro:if value="${count != len(axes)}">
+          <link name="test_rail_link_${count}"/>
+        </xacro:if>
+        <xacro:if value="${count == 1}">
+          <!-- <link name="test_rail_link_1"/> -->
+          <xacro:property name="joint_child" value="test_rail_carriage"/>
+        </xacro:if>
+        <xacro:if value="${axes[count - 1] == 'x'}">
+          <xacro:property name="axis_control" value="1 0 0"/>
+          <xacro:property name="lower_limit" value="${test_rail_config['x_axis_limits'][0]}"/>
+          <xacro:property name="upper_limit" value="${test_rail_config['x_axis_limits'][1]}"/>
+        </xacro:if>
+        <xacro:if value="${axes[count - 1]  == 'y'}">
+          <xacro:property name="axis_control" value="0 1 0"/>
+          <xacro:property name="lower_limit" value="${test_rail_config['y_axis_limits'][0]}"/>
+          <xacro:property name="upper_limit" value="${test_rail_config['y_axis_limits'][1]}"/>
+        </xacro:if>
+        <xacro:if value="${axes[count - 1] == 'z'}">
+          <xacro:property name="axis_control" value="0 0 1"/>
+          <xacro:property name="lower_limit" value="${test_rail_config['z_axis_limits'][0]}"/>
+          <xacro:property name="upper_limit" value="${test_rail_config['z_axis_limits'][1]}"/>
+        </xacro:if>
+        <joint name="test_rail_joint_${count}" type="prismatic">
+          <parent link="${joint_parent}"/>
+          <child link="${joint_child}"/>
+          <axis xyz="${axis_control}"/>
+          <origin xyz="0 0 0" rpy="0 0 0"/>
+          <limit lower="${lower_limit}" upper="${upper_limit}" effort="1000.0" velocity="0.5"/>
+          <dynamics damping="10.0" friction="1.0"/>
+        </joint>
+      </xacro:if>
+    </xacro:macro>
     <joint name="${parent}_to_test_rail" type="fixed">
       <parent link="${parent}"/>
@@ -14,5 +58,5 @@
       <visual>
         <geometry>
-          <box size="${rail_rail_config['rail_length']} ${rail_rail_config['rail_width']} 0.1"/>
+          <box size="${test_rail_config['rail_length']} ${test_rail_config['rail_width']} ${test_rail_config['rail_height']}"/>
         </geometry>
         <material name="grey"><color rgba="0.5 0.5 0.5 1.0"/></material>
@@ -31,4 +75,5 @@
       </inertial>
     </link>
+    <xacro:build_joints count="${len(axes)}"/>
     <link name="test_rail_carriage">
       <visual>
@@ -44,11 +89,5 @@
       </collision> -->
     </link>
-    <joint name="test_rail_joint" type="prismatic">
-      <parent link="test_rail_base"/>
-      <child link="test_rail_carriage"/>
-      <axis xyz="1 0 0"/>
-      <limit lower="${-0.5 * rail_rail_config['rail_length']}" upper="${0.5 * rail_rail_config['rail_length']}" effort="1000.0" velocity="0.5"/>
-      <dynamics damping="10.0" friction="1.0"/>
-    </joint>
+    <xacro:test_rail_ros2_control num_axes="${len(test_rail_config['axes'])}"/>
   </xacro:macro>
 </robot>
